File: elec/hw/cartes/pmi_2023/pmi_2023.kicad_sch (KiCad schematic)
At the start: 5 parts, among them U1 STM32F401RBTx

Commit message: pmi_2023 schematics
Parts:
- removed R1, R2, R3, R4: R, symbol Device:R
- removed U1: STM32F401RBTx, Package_QFP:LQFP-64_10x10mm_P0.5mm, symbol MCU_ST_STM32F4:STM32F401RBTx
Other:
- added sheet actuators (actuators.kicad_sch)
- added sheet com (com.kicad_sch)
- added sheet power_supply (power_supply.kicad_sch)
- added sheet propulsion (propulsion.kicad_sch)
- added sheet sensors (sensors.kicad_sch)
- added sheet uc (uc.kicad_sch)

Commit message: pmi 2023 wip
Other:
- removed sheet uc
- sheet actuators ports: added LED_RGB_B_3v3, LED_RGB_G_3v3, LED_RGB_R_3v3, LED_RGB_W_3v3, enable_tof_3v3, line_led_pwm_3v3, scl_3v3, sda_3v3, /reset_tof_3v3; removed none
- sheet com ports: added dir_left, dir_right, left_encod_A_3v3, left_encod_B_3v3, pwm_left, pwm_right, pwm_vaccum_3v3, right_encod_A_3v3, right_encod_B_3v3; removed esp32_miso_3v3, esp32_mosi_3v3, esp32_ncs_3v3, esp32_sck_3v3
- sheet sensors ports: added none; removed line_detect_center
- note added: "ajouter KTS1622EUAA-TR pour 16 io"

Commit message: pmi2023 wip
Other:
- added sheet interface (interface.kicad_sch)
- sheet actuators ports: added pwm_vaccum_3v3; removed none
- sheet com ports: added ctc_left, ctc_right, gyro_miso_3v3, gyro_mosi_3v3, gyro_ncs_3v3, gyro_sck_3v3, i2C_io_int_3v3, i_prop_left_3v3, i_prop_right_3v3, scl_3v3, sda_3v3, tof_irq; removed esp32_scl_3v3, esp32_sda_3v3, pwm_vaccum_3v3
- sheet sensors ports: added ctc_left, ctc_right, gyro_miso_3v3, gyro_mosi_3v3, gyro_ncs_3v3, gyro_sck_3v3, tof_irq; removed ctc_front_left, ctc_front_rigth, ctc_rear_left, ctc_rear_right, tof_irq[0..7]
- note removed: "ajouter KTS1622EUAA-TR pour 16 io"

Commit message: pmi2023 wip
Changed lines of the file:
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@@
-    (stroke (width 0) (type default))
-  )
-  (wire (pts (xy 138.43 54.61) (xy 138.43 46.99))
     (stroke (width 0) (type default))
   )
@@
     (stroke (width 0) (type default))
   )
-  (wire (pts (xy 69.85 54.61) (xy 138.43 54.61))
+  (wire (pts (xy 69.85 46.99) (xy 220.98 46.99))
     (stroke (width 0) (type default))
   )
@@
     (stroke (width 0) (type default))
   )
-  (wire (pts (xy 210.82 52.07) (xy 220.98 52.07))
+  (wire (pts (xy 210.82 54.61) (xy 220.98 54.61))
     (stroke (width 0) (type default))
   )
@@
     (stroke (width 0) (type default))
   )
-  (wire (pts (xy 210.82 58.42) (xy 220.98 58.42))
+  (wire (pts (xy 210.82 60.96) (xy 220.98 60.96))
     (stroke (width 0) (type default))
   )
@@
     (stroke (width 0) (type default))
   )
-  (wire (pts (xy 210.82 54.61) (xy 220.98 54.61))
+  (wire (pts (xy 210.82 57.15) (xy 220.98 57.15))
     (stroke (width 0) (type default))
   )
@@
     (stroke (width 0) (type default))
   )
-  (wire (pts (xy 138.43 46.99) (xy 220.98 46.99))
-    (stroke (width 0) (type default))
-  )
   (wire (pts (xy 139.7 105.41) (xy 157.48 105.41))
     (stroke (width 0) (type default))
@@
     (stroke (width 0) (type default))
   )
-  (wire (pts (xy 210.82 60.96) (xy 220.98 60.96))
+  (wire (pts (xy 210.82 63.5) (xy 220.98 63.5))
     (stroke (width 0) (type default))
   )
@@
     (effects (font (size 1.27 1.27)) (justify left bottom))
   )
-  (sheet (at 15.24 19.05) (size 19.05 24.13) (fields_autoplaced)
+  (sheet (at 223.52 101.6) (size 53.34 25.4) (fields_autoplaced)
     (stroke (width 0.1524) (type solid))
     (fill (color 160 255 127 1.0000))
-    (property "Sheetname" "power_supply" (at 15.24 18.3384 0)
+    (property "Sheetname" "power_supply" (at 223.52 100.8884 0)
       (effects (font (size 1.27 1.27)) (justify left bottom))
     )
-    (property "Sheetfile" "power_supply.kicad_sch" (at 15.24 43.7646 0)
+    (property "Sheetfile" "power_supply.kicad_sch" (at 223.52 127.5846 0)
       (effects (font (size 1.27 1.27)) (justify left top))
     )
@@
     )
   )
-  (sheet (at 38.1 50.8) (size 31.75 92.71) (fields_autoplaced)
+  (sheet (at 38.1 40.64) (size 31.75 102.87) (fields_autoplaced)
     (stroke (width 0.1524) (type solid))
     (fill (color 160 255 127 1.0000))
-    (property "Sheetname" "actuators" (at 38.1 50.0884 0)
+    (property "Sheetname" "actuators" (at 38.1 39.9284 0)
       (effects (font (size 1.27 1.27)) (justify left bottom))
     )
@@
       (effects (font (size 1.27 1.27)) (justify right))
     )
-    (pin "pwm_vaccum_3v3" output (at 69.85 54.61 0)
+    (pin "pwm_vaccum_3v3" output (at 69.85 46.99 0)
       (effects (font (size 1.27 1.27)) (justify right))
     )
@@
       (effects (font (size 1.27 1.27)) (justify right))
     )
-    (pin "vbatt_mon_8.7V" output (at 157.48 53.34 180)
-      (effects (font (size 1.27 1.27)) (justify left))
+    (pin "vbatt_mon_8.7V" input (at 210.82 110.49 0)
+      (effects (font (size 1.27 1.27)) (justify right))
     )
     (pin "esp32_tx2_3v3" output (at 187.96 49.53 90)
@@
       (effects (font (size 1.27 1.27)) (justify right))
     )
-    (pin "pwm_left" output (at 210.82 52.07 0)
-      (effects (font (size 1.27 1.27)) (justify right))
-    )
-    (pin "pwm_right" output (at 210.82 60.96 0)
-      (effects (font (size 1.27 1.27)) (justify right))
-    )
-    (pin "dir_right" output (at 210.82 58.42 0)
-      (effects (font (size 1.27 1.27)) (justify right))
-    )
-    (pin "dir_left" output (at 210.82 54.61 0)
+    (pin "pwm_left" output (at 210.82 54.61 0)
+      (effects (font (size 1.27 1.27)) (justify right))
+    )
+    (pin "pwm_right" output (at 210.82 63.5 0)
+      (effects (font (size 1.27 1.27)) (justify right))
+    )
+    (pin "dir_right" output (at 210.82 60.96 0)
+      (effects (font (size 1.27 1.27)) (justify right))
+    )
+    (pin "dir_left" output (at 210.82 57.15 0)
       (effects (font (size 1.27 1.27)) (justify right))
     )
@@
       (effects (font (size 1.27 1.27)) (justify left top))
     )
-    (pin "pwm_left" input (at 220.98 52.07 180)
-      (effects (font (size 1.27 1.27)) (justify left))
-    )
-    (pin "dir_left" input (at 220.98 54.61 180)
-      (effects (font (size 1.27 1.27)) (justify left))
-    )
-    (pin "pwm_right" input (at 220.98 58.42 180)
-      (effects (font (size 1.27 1.27)) (justify left))
-    )
-    (pin "dir_right" input (at 220.98 60.96 180)
-      (effects (font (size 1.27 1.27)) (justify left))
-    )
+    (pin "pwm_left" input (at 220.98 54.61 180)
+      (effects (font (size 1.27 1.27)) (justify left))
+    )
+    (pin "dir_left" input (at 220.98 57.15 180)
+      (effects (font (size 1.27 1.27)) (justify left))
+    )
+    (pin "pwm_right" input (at 220.98 60.96 180)
+      (effects (font (size 1.27 1.27)) (justify left))
+    )
+    (pin "dir_right" input (at 220.98 63.5 180)
+      (effects (font (size 1.27 1.27)) (justify left))
+    )

Commit message: wip
Other:
- sheet com ports: added vbatt_mon_4.35V; removed vbatt_mon_8.7V
- sheet power_supply ports: added vbatt_mon_4.35V; removed none
Changed lines of the file:
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@@
+    (stroke (width 0) (type default))
+  )
+  (wire (pts (xy 210.82 110.49) (xy 223.52 110.49))
     (stroke (width 0) (type default))
   )
@@
     (property "Sheetfile" "power_supply.kicad_sch" (at 223.52 127.5846 0)
       (effects (font (size 1.27 1.27)) (justify left top))
+    )
+    (pin "vbatt_mon_4.35V" output (at 223.52 110.49 180)
+      (effects (font (size 1.27 1.27)) (justify left))
     )
     (instances
@@
       (effects (font (size 1.27 1.27)) (justify right))
     )
-    (pin "vbatt_mon_8.7V" input (at 210.82 110.49 0)
-      (effects (font (size 1.27 1.27)) (justify right))
-    )
+    (pin "vbatt_mon_4.35V" input (at 210.82 110.49 0)
+      (effects (font (size 1.27 1.27)) (justify right))
+    )

Commit message: wip
Other:
- sheet power_supply ports: added Vmot_left_5V, Vmot_right_5V, enable_pw_conv_3v7; removed none
Changed lines of the file:
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@@
+      (effects (font (size 1.27 1.27)) (justify left))
+    )
+    (pin "Vmot_left_5V" output (at 276.86 105.41 0)
+      (effects (font (size 1.27 1.27)) (justify right))
+    )
+    (pin "Vmot_right_5V" output (at 276.86 107.95 0)
+      (effects (font (size 1.27 1.27)) (justify right))
+    )
+    (pin "enable_pw_conv_3v7" output (at 223.52 113.03 180)
       (effects (font (size 1.27 1.27)) (justify left))
     )

Commit message: wip
Parts:
- added H1, H2, H3, H4: MountingHole, MountingHole:MountingHole_2.1mm, symbol Mechanical:MountingHole
Changed lines of the file:
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@@
     (effects (font (size 1.27 1.27)) (justify left bottom))
+  )
+  (symbol (lib_id "Mechanical:MountingHole") (at 120.65 181.61 0) (unit 1)
+    (in_bom yes) (on_board yes) (dnp no) (fields_autoplaced)
+    (property "Reference" "H4" (at 123.19 180.34 0)
+      (effects (font (size 1.27 1.27)) (justify left))
+    )
+    (property "Value" "MountingHole" (at 123.19 182.88 0)
+      (effects (font (size 1.27 1.27)) (justify left))
+    )
+    (property "Footprint" "MountingHole:MountingHole_2.1mm" (at 120.65 181.61 0)
+      (effects (font (size 1.27 1.27)) hide)
+    )
+    (property "Datasheet" "~" (at 120.65 181.61 0)
+      (effects (font (size 1.27 1.27)) hide)
+    )
+    (instances
+      (project "pmi_2023"
+        (path "/334a657f-c66c-4260-9567-14f1c99913d7"
+          (reference "H4") (unit 1)
+        )
+      )
+    )
+  )
+  (symbol (lib_id "Mechanical:MountingHole") (at 120.65 172.72 0) (unit 1)
+    (in_bom yes) (on_board yes) (dnp no) (fields_autoplaced)
+    (property "Reference" "H2" (at 123.19 171.45 0)
+      (effects (font (size 1.27 1.27)) (justify left))
+    )
+    (property "Value" "MountingHole" (at 123.19 173.99 0)
+      (effects (font (size 1.27 1.27)) (justify left))
+    )
+    (property "Footprint" "MountingHole:MountingHole_2.1mm" (at 120.65 172.72 0)
+      (effects (font (size 1.27 1.27)) hide)
+    )
+    (property "Datasheet" "~" (at 120.65 172.72 0)
+      (effects (font (size 1.27 1.27)) hide)
+    )
+    (instances
+      (project "pmi_2023"
+        (path "/334a657f-c66c-4260-9567-14f1c99913d7"
+          (reference "H2") (unit 1)
+        )
+      )
+    )
+  )
+  (symbol (lib_id "Mechanical:MountingHole") (at 97.79 172.72 0) (unit 1)
+    (in_bom yes) (on_board yes) (dnp no) (fields_autoplaced)
+    (property "Reference" "H1" (at 100.33 171.45 0)
+      (effects (font (size 1.27 1.27)) (justify left))
+    )
+    (property "Value" "MountingHole" (at 100.33 173.99 0)
+      (effects (font (size 1.27 1.27)) (justify left))
+    )
+    (property "Footprint" "MountingHole:MountingHole_2.1mm" (at 97.79 172.72 0)
+      (effects (font (size 1.27 1.27)) hide)
+    )
+    (property "Datasheet" "~" (at 97.79 172.72 0)
+      (effects (font (size 1.27 1.27)) hide)
+    )
+    (instances
+      (project "pmi_2023"
+        (path "/334a657f-c66c-4260-9567-14f1c99913d7"
+          (reference "H1") (unit 1)
+        )
+      )
+    )
+  )
+  (symbol (lib_id "Mechanical:MountingHole") (at 97.79 181.61 0) (unit 1)
+    (in_bom yes) (on_board yes) (dnp no) (fields_autoplaced)
+    (property "Reference" "H3" (at 100.33 180.34 0)
+      (effects (font (size 1.27 1.27)) (justify left))
+    )
+    (property "Value" "MountingHole" (at 100.33 182.88 0)
+      (effects (font (size 1.27 1.27)) (justify left))
+    )
+    (property "Footprint" "MountingHole:MountingHole_2.1mm" (at 97.79 181.61 0)
+      (effects (font (size 1.27 1.27)) hide)
+    )
+    (property "Datasheet" "~" (at 97.79 181.61 0)
+      (effects (font (size 1.27 1.27)) hide)
+    )
+    (instances
+      (project "pmi_2023"
+        (path "/334a657f-c66c-4260-9567-14f1c99913d7"
+          (reference "H3") (unit 1)
+        )
+      )
+    )
   )
   (sheet (at 223.52 101.6) (size 53.34 25.4) (fields_autoplaced)
