File: elec/hw/cartes/pmi_2023/sensors.kicad_sch (KiCad schematic)
At the start: 48 parts, among them U10 AD8531ARTZ, U11 GP2S60B, U12 GP2S60B, U13 GP2S60B, U14 GP2S60B, U15 GP2S60B, U16 GP2S60B, U17 GP2S60B, U18 GP2S60B, U19 tof_sensor_master, U20 tof_sensor_master, U21 tof_sensor_master, U22 tof_sensor_master, U23 tof_sensor_master, U24 tof_sensor_master, U25 tof_sensor_master, U26 tof_sensor_master, U27 GP2S60B

Commit message: pmi 2023 wip
Parts:
- removed R83, R84: 100k, cocotter_resistor:r0603_reflow, symbol cocotter_resistors:R_100k_0603_1%
- removed R85: 150R 1%, symbol cocotter_resistors:R_150R_0805_1%
- removed R86: 27k 1%, cocotter_resistor:r0603_reflow, symbol cocotter_resistors:R_27k_0603_1%
- removed U27: GP2S60B, symbol cocotter_ic:GP2S60B
Connections:
- net ctc_rear_left is gone; now on net ctc_left: SW_RL.1, SW_RL.2
- net ctc_rear_right is gone; now on net ctc_rigth: SW_RR.3, SW_RR.4
- net ctc_front_left renamed ctc_left
- net ctc_front_rigth renamed ctc_rigth

Commit message: pmi2023 wip
Parts:
- added C23: 100nF 50V, symbol cocotter_capacitors:C_100nF_50V_0603
- added R53, R54, R55, R56: 100k, cocotter_resistor:r0603_reflow, symbol cocotter_resistors:R_100k_0603_1%
- added U9: ~, symbol cocotter_ic:LSM6DSO32XTR
Connections:
- net tof_irq1 is gone; now on net tof_irq: U20.4 (detect_irq_3v3)
- net tof_irq2 is gone; now on net tof_irq: U21.4 (detect_irq_3v3)
- net tof_irq3 is gone; now on net tof_irq: U22.4 (detect_irq_3v3)
- net tof_irq4 is gone; now on net tof_irq: U23.4 (detect_irq_3v3)
- net tof_irq5 is gone; now on net tof_irq: U24.4 (detect_irq_3v3)
- net tof_irq6 is gone; now on net tof_irq: U25.4 (detect_irq_3v3)
- net tof_irq7 is gone; now on net tof_irq: U26.4 (detect_irq_3v3)
- net +3.3V: now also C23.1, R53.1, R54.1, R55.1, R56.1, U9.5 (Vdd_IO), U9.8 (Vdd)
- net GND: now also C23.2, U9.6 (GND), U9.7 (GND)
- net tof_irq0 renamed tof_irq
- new net: R53.2, U9.3 (SCx)
- new net: R56.2, U9.4 (INT1)
- new net: R54.2, U9.2 (SDx)
- new net gyro_miso_3v3: U9.1 (SDO)
- new net gyro_mosi_3v3: U9.12 (SDA/SDI)
- new net gyro_ncs_3v3: R55.2, U9.12 (SDA/SDI)
- new net gyro_sck_3v3: U9.13 (SCL/SCK)
Other:
- note removed: "tof_irq[0..7]"
- moved on the sheet: R81, R82, SW_FL, SW_FR, SW_RL, SW_RR, U19, U20, U21, U22, U23, U24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

Commit message: pmi_2023 wip
Parts:
- C23, C24, C26: footprint (none) -> cocotter_capacitors:C_0603_1608Metric
- C25: footprint (none) -> cocotter_capacitors:C_0805_2012Metric
- R65, R67, R69, R71, R73, R75, R77, R79: footprint (none) -> cocotter_resistor:r0805_reflow
- U10: footprint (none) -> cocotter_ic:SOT23-5
- U11, U12, U13, U14, U15, U16, U17, U18: footprint (none) -> cocotter_ic:GP2S60
- U19, U20, U21, U22, U23, U24, U25, U26: footprint (none) -> cocotter_connectors:tof_sensor_male
- U9: footprint (none) -> cocotter_ic:LGA-14_3x2.5mm_P0.5mm_LayoutBorder3x4y
- renumbered SW_FL to SW_FL1, SW_FR to SW_FR1, SW_RL to SW_RL1, SW_RR to SW_RR1
Changed lines of the file:
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@@
   (symbol (lib_id "cocotter_connectors:SPVT210104") (at 73.66 189.23 180) (unit 1)
     (in_bom yes) (on_board yes) (dnp no)
-    (property "Reference" "SW_RR" (at 73.66 195.58 0)
+    (property "Reference" "SW_RR1" (at 73.66 195.58 0)
       (effects (font (size 1.27 1.27)))
     )
@@
       (project "pmi_2023"
         (path "/334a657f-c66c-4260-9567-14f1c99913d7/7e29bdf2-f1b2-4a04-a6a0-e1a9d40b2651"
-          (reference "SW_RR") (unit 1)
+          (reference "SW_RR1") (unit 1)
         )
       )
@@
   (symbol (lib_id "cocotter_connectors:SPVT110106") (at 33.02 189.23 180) (unit 1)
     (in_bom yes) (on_board yes) (dnp no)
-    (property "Reference" "SW_RL" (at 33.02 195.58 0)
+    (property "Reference" "SW_RL1" (at 33.02 195.58 0)
       (effects (font (size 1.27 1.27)))
     )
@@
       (project "pmi_2023"
         (path "/334a657f-c66c-4260-9567-14f1c99913d7/7e29bdf2-f1b2-4a04-a6a0-e1a9d40b2651"
-          (reference "SW_RL") (unit 1)
+          (reference "SW_RL1") (unit 1)
         )
       )
@@
       (effects (font (size 1.27 1.27)))
     )
-    (property "Footprint" "" (at 101.6 53.34 0)
+    (property "Footprint" "cocotter_ic:GP2S60" (at 101.6 53.34 0)
       (effects (font (size 1.27 1.27)) hide)
     )
@@
       (effects (font (size 1.27 1.27)) (justify left))
     )
-    (property "Footprint" "" (at 58.1152 26.67 0)
+    (property "Footprint" "cocotter_capacitors:C_0603_1608Metric" (at 58.1152 26.67 0)
       (effects (font (size 1.27 1.27)) hide)
     )
@@
       (effects (font (size 1.27 1.27)) (justify left))
     )
-    (property "Footprint" "" (at 172.4152 167.64 0)
+    (property "Footprint" "cocotter_capacitors:C_0603_1608Metric" (at 172.4152 167.64 0)
       (effects (font (size 1.27 1.27)) hide)
     )
@@
       (effects (font (size 1.27 1.27)))
     )
-    (property "Footprint" "" (at 223.012 83.82 0)
+    (property "Footprint" "cocotter_connectors:tof_sensor_male" (at 223.012 83.82 0)
       (effects (font (size 1.27 1.27)) hide)
     )
@@
       (effects (font (size 1.27 1.27)))
     )
-    (property "Footprint" "" (at 162.052 127 0)
+    (property "Footprint" "cocotter_connectors:tof_sensor_male" (at 162.052 127 0)
       (effects (font (size 1.27 1.27)) hide)
     )
@@
   (symbol (lib_id "cocotter_connectors:SPVT210104") (at 33.02 172.72 0) (unit 1)
     (in_bom yes) (on_board yes) (dnp no)
-    (property "Reference" "SW_FL" (at 33.02 167.64 0)
+    (property "Reference" "SW_FL1" (at 33.02 167.64 0)
       (effects (font (size 1.27 1.27)))
     )
@@
       (project "pmi_2023"
         (path "/334a657f-c66c-4260-9567-14f1c99913d7/7e29bdf2-f1b2-4a04-a6a0-e1a9d40b2651"
-          (reference "SW_FL") (unit 1)
+          (reference "SW_FL1") (unit 1)
         )
       )
@@
       (effects (font (size 1.27 1.27)))
     )
-    (property "Footprint" "" (at 140.97 27.94 0)
+    (property "Footprint" "cocotter_ic:GP2S60" (at 140.97 27.94 0)
       (effects (font (size 1.27 1.27)) hide)
     )
@@
       (effects (font (size 1.27 1.27)) (justify left))
     )
-    (property "Footprint" "" (at 206.502 21.59 90)
+    (property "Footprint" "cocotter_resistor:r0805_reflow" (at 206.502 21.59 90)
       (effects (font (size 1.27 1.27)) hide)
     )
@@
       (effects (font (size 1.27 1.27)))
     )
-    (property "Footprint" "" (at 219.71 53.34 0)
+    (property "Footprint" "cocotter_ic:GP2S60" (at 219.71 53.34 0)
       (effects (font (size 1.27 1.27)) hide)
     )
@@
       (effects (font (size 1.27 1.27)))
     )
-    (property "Footprint" "" (at 162.052 83.82 0)
+    (property "Footprint" "cocotter_connectors:tof_sensor_male" (at 162.052 83.82 0)
       (effects (font (size 1.27 1.27)) hide)
     )
@@
       (effects (font (size 1.27 1.27)) (justify left))
     )
-    (property "Footprint" "" (at 74.6252 26.67 0)
+    (property "Footprint" "cocotter_capacitors:C_0805_2012Metric" (at 74.6252 26.67 0)
       (effects (font (size 1.27 1.27)) hide)
     )
@@
       (effects (font (size 1.27 1.27)))
     )
-    (property "Footprint" "" (at 219.71 27.94 0)
+    (property "Footprint" "cocotter_ic:GP2S60" (at 219.71 27.94 0)
       (effects (font (size 1.27 1.27)) hide)
     )
@@
       (effects (font (size 1.27 1.27)))
     )
-    (property "Footprint" "" (at 101.092 83.82 0)
+    (property "Footprint" "cocotter_connectors:tof_sensor_male" (at 101.092 83.82 0)
       (effects (font (size 1.27 1.27)) hide)
     )
@@
       (effects (font (size 1.27 1.27)) (justify left))
     )
-    (property "Footprint" "" (at 127.762 46.99 90)
+    (property "Footprint" "cocotter_resistor:r0805_reflow" (at 127.762 46.99 90)
       (effects (font (size 1.27 1.27)) hide)
     )
@@
       (effects (font (size 1.27 1.27)))
     )
-    (property "Footprint" "" (at 140.97 53.34 0)
+    (property "Footprint" "cocotter_ic:GP2S60" (at 140.97 53.34 0)
       (effects (font (size 1.27 1.27)) hide)
     )
@@
       (effects (font (size 1.27 1.27)) (justify left))
     )
-    (property "Footprint" "" (at 88.392 21.59 90)
+    (property "Footprint" "cocotter_resistor:r0805_reflow" (at 88.392 21.59 90)
       (effects (font (size 1.27 1.27)) hide)
     )
@@
       (effects (font (size 1.27 1.27)) (justify left))
     )
-    (property "Footprint" "" (at 33.9852 39.37 0)
+    (property "Footprint" "cocotter_capacitors:C_0603_1608Metric" (at 33.9852 39.37 0)
       (effects (font (size 1.27 1.27)) hide)
     )
@@
       (effects (font (size 1.27 1.27)) (justify left))
     )
-    (property "Footprint" "" (at 167.132 46.99 90)
+    (property "Footprint" "cocotter_resistor:r0805_reflow" (at 167.132 46.99 90)
       (effects (font (size 1.27 1.27)) hide)
     )
@@
       (effects (font (size 1.27 1.27)))
     )
-    (property "Footprint" "" (at 223.012 127 0)
+    (property "Footprint" "cocotter_connectors:tof_sensor_male" (at 223.012 127 0)
       (effects (font (size 1.27 1.27)) hide)
     )
@@
       (effects (font (size 1.27 1.27)) (justify left))
     )
-    (property "Footprint" "" (at 206.502 46.99 90)
+    (property "Footprint" "cocotter_resistor:r0805_reflow" (at 206.502 46.99 90)
       (effects (font (size 1.27 1.27)) hide)
     )
@@
       (effects (font (size 1.27 1.27)))
     )
-    (property "Footprint" "" (at 101.6 27.94 0)
+    (property "Footprint" "cocotter_ic:GP2S60" (at 101.6 27.94 0)
       (effects (font (size 1.27 1.27)) hide)
     )
@@
       (effects (font (size 1.27 1.27)))
     )
-    (property "Footprint" "" (at 52.07 33.02 0)
+    (property "Footprint" "cocotter_ic:SOT23-5" (at 52.07 33.02 0)
       (effects (font (size 1.27 1.27)) hide)
     )
@@
       (effects (font (size 1.27 1.27)))
     )
-    (property "Footprint" "" (at 101.092 127 0)
+    (property "Footprint" "cocotter_connectors:tof_sensor_male" (at 101.092 127 0)
       (effects (font (size 1.27 1.27)) hide)
     )
@@
       (effects (font (size 1.27 1.27)))
     )
-    (property "Footprint" "" (at 143.51 171.45 0)
+    (property "Footprint" "cocotter_ic:LGA-14_3x2.5mm_P0.5mm_LayoutBorder3x4y" (at 143.51 171.45 0)
       (effects (font (size 1.27 1.27)) hide)
     )
@@
       (effects (font (size 1.27 1.27)) (justify left))
     )
-    (property "Footprint" "" (at 88.392 46.99 90)
+    (property "Footprint" "cocotter_resistor:r0805_reflow" (at 88.392 46.99 90)
       (effects (font (size 1.27 1.27)) hide)
     )
@@
       (effects (font (size 1.27 1.27)))
     )
-    (property "Footprint" "" (at 180.34 27.94 0)
+    (property "Footprint" "cocotter_ic:GP2S60" (at 180.34 27.94 0)
       (effects (font (size 1.27 1.27)) hide)
     )
@@
       (effects (font (size 1.27 1.27)))
     )
-    (property "Footprint" "" (at 40.132 83.82 0)
+    (property "Footprint" "cocotter_connectors:tof_sensor_male" (at 40.132 83.82 0)
       (effects (font (size 1.27 1.27)) hide)
     )
@@
       (effects (font (size 1.27 1.27)))
     )
-    (property "Footprint" "" (at 180.34 53.34 0)
+    (property "Footprint" "cocotter_ic:GP2S60" (at 180.34 53.34 0)
       (effects (font (size 1.27 1.27)) hide)
     )
@@
       (effects (font (size 1.27 1.27)) (justify left))
     )
-    (property "Footprint" "" (at 167.132 21.59 90)
+    (property "Footprint" "cocotter_resistor:r0805_reflow" (at 167.132 21.59 90)
       (effects (font (size 1.27 1.27)) hide)
     )
@@
   (symbol (lib_id "cocotter_connectors:SPVT110106") (at 73.66 172.72 0) (unit 1)
     (in_bom yes) (on_board yes) (dnp no)
-    (property "Reference" "SW_FR" (at 73.66 167.64 0)
+    (property "Reference" "SW_FR1" (at 73.66 167.64 0)
       (effects (font (size 1.27 1.27)))
     )
@@
       (project "pmi_2023"
         (path "/334a657f-c66c-4260-9567-14f1c99913d7/7e29bdf2-f1b2-4a04-a6a0-e1a9d40b2651"
-          (reference "SW_FR") (unit 1)
+          (reference "SW_FR1") (unit 1)
         )
       )
@@
       (effects (font (size 1.27 1.27)))
     )
-    (property "Footprint" "" (at 40.132 127 0)
+    (property "Footprint" "cocotter_connectors:tof_sensor_male" (at 40.132 127 0)
       (effects (font (size 1.27 1.27)) hide)
     )
@@
       (effects (font (size 1.27 1.27)) (justify left))
     )
-    (property "Footprint" "" (at 127.762 21.59 90)
-      (effects (font (size 1.27 1.27)) hide)
-    )
+    (property "Footprint" "cocotter_resistor:r0805_reflow" (at 127.762 21.59 90)
+      (effects (font (size 1.27 1.27)) hide)
+    )

Commit message: wip
Parts:
- added R109: 100k, cocotter_resistor:r0603_reflow, symbol cocotter_resistors:R_100k_0603_1%
- C10: renamed from C26; JLCPCB (none) -> C14663
- C11: renamed from C25; value 10µF 16V -> 10µF 25V; symbol cocotter_capacitors:C_10µF_16V_0805 -> cocotter_capacitors:C_10µF_16V_0805_X5R; JLCPCB (none) -> C15850; Specification 10µF 16V X7R 0805 -> 10µF 25V X5R 0805
- C12: renamed from C23; JLCPCB (none) -> C14663
- C9: renamed from C24; JLCPCB (none) -> C14663
- R31: renamed from R64; JLCPCB (none) -> C25803
- R32: renamed from R81; JLCPCB (none) -> C25803
- R33: renamed from R82; JLCPCB (none) -> C25803
- R34: renamed from R65; JLCPCB (none) -> C17471
- R35: renamed from R73; JLCPCB (none) -> C17471
- R36: renamed from R66; JLCPCB (none) -> C22967; mouser 603-RC0603FR-10100KL -> (none)
- R37: renamed from R74; JLCPCB (none) -> C22967; mouser 603-RC0603FR-10100KL -> (none)
- R38: renamed from R56; JLCPCB (none) -> C25803
- R39: renamed from R55; JLCPCB (none) -> C25803
- R40: renamed from R67; JLCPCB (none) -> C17471
- R41: renamed from R75; JLCPCB (none) -> C17471
- R42: renamed from R68; JLCPCB (none) -> C22967; mouser 603-RC0603FR-10100KL -> (none)
- R43: renamed from R76; JLCPCB (none) -> C22967; mouser 603-RC0603FR-10100KL -> (none)
- R44: renamed from R53; JLCPCB (none) -> C25803
- R45: renamed from R54; JLCPCB (none) -> C25803
- R46: renamed from R69; JLCPCB (none) -> C17471
- R47: renamed from R77; JLCPCB (none) -> C17471
- R48: renamed from R70; JLCPCB (none) -> C22967; mouser 603-RC0603FR-10100KL -> (none)
- R49: renamed from R78; JLCPCB (none) -> C22967; mouser 603-RC0603FR-10100KL -> (none)
- R50: renamed from R71; JLCPCB (none) -> C17471
- R51: renamed from R79; JLCPCB (none) -> C17471
- R52: renamed from R72; JLCPCB (none) -> C22967; mouser 603-RC0603FR-10100KL -> (none)
- R53: renamed from R80; JLCPCB (none) -> C22967; mouser 603-RC0603FR-10100KL -> (none)
- SW2: renamed from SW_RL1; value ~ -> SPVT110106
- SW3: renamed from SW_FR1; value ~ -> SPVT110106
- U12: renamed from U9; value ~ -> LSM6DSO32XTR; JLCPCB (none) -> C2655100
- U13: renamed from U12; JLCPCB (none) -> C83485
- U14: renamed from U16; JLCPCB (none) -> C83485
- U15: renamed from U13; JLCPCB (none) -> C83485
- U16: renamed from U17; JLCPCB (none) -> C83485
- U19: renamed from U14; JLCPCB (none) -> C83485
- U20: renamed from U18; JLCPCB (none) -> C83485
- U5: renamed from U10; JLCPCB (none) -> C143905
- U8: renamed from U11; JLCPCB (none) -> C83485
- U9: renamed from U15; JLCPCB (none) -> C83485
- renumbered SW_FL1 to SW1, SW_RR1 to SW4, U20 to U10, U24 to U11, U21 to U17, U25 to U18, U22 to U21, U26 to U22, U19 to U6, U23 to U7
Connections:
- net +3.3V: now also R109.1
- net gyro_mosi_3v3: now also U12.14 (SDA/SDI); no longer U12.12 (SDA/SDI)
- net at U12.4 (INT1): now also R109.2; no longer R38.2
- net at U12.9 (INT2/DEN): now also R38.2
Other:
- note added: "TODO gerer IRQ"
- moved on the sheet: C12, R32, R33, R38, R39, R44, R45, SW1, SW2, SW3, SW4, U12

Commit message: wip
Parts:
- removed SW1, SW4: SPVT210104, symbol cocotter_connectors:SPVT210104
- removed SW2, SW3: SPVT110106, symbol cocotter_connectors:SPVT110106
- removed U11, U18, U22, U7: tof_sensor_master, cocotter_connectors:tof_sensor_male, symbol cocotter_connectors:tof_sensor_master
- added C47: 100nF 50V, cocotter_capacitors:C_0603_1608Metric, symbol cocotter_capacitors:C_100nF_50V_0603
- added C48: 10µF 25V, cocotter_capacitors:C_0805_2012Metric, symbol cocotter_capacitors:C_10µF_16V_0805_X5R
- added R10, R11, R12: 0R, cocotter_resistor:r0603_reflow, symbol cocotter_resistors:R_0R_0603
- added R9: 100k, cocotter_resistor:r0603_reflow, symbol cocotter_resistors:R_100k_0603_1%
- added SW1: ESE22MH22, cocotter_connectors:ESE22MH22, symbol cocotter_connectors:ESE22MH22
- added SW2: ESE22MH24, cocotter_connectors:ESE22MH24, symbol cocotter_connectors:ESE22MH24
- added U7: XRA1200PIG16TR-F, cocotter_ic:TSSOP-16_4.4x5mm_P0.65mm, symbol cocotter_ic:XRA1200PIG16TR-F
- U5: footprint cocotter_ic:SOT23-5 -> cocotter_ic:SOT-23-5
Connections:
- net +3.3V: now also C47.1, C48.1, R9.1, U7.16 (VCC)
- net GND: now also C47.2, C48.2, R10.2, R11.2, R12.2, SW1.1, SW2.2, U7.8 (GND)
- net ctc_left: now also SW1.2
- net ctc_rigth: now also SW2.1
- net line_detect_l0: now also U7.4 (P0)
- net line_detect_l1: now also U7.5 (P1)
- net line_detect_l2: now also U7.6 (P2)
- net line_detect_l3: now also U7.7 (P3)
- net line_detect_r0: now also U7.9 (P4)
- net line_detect_r1: now also U7.10 (P5)
- net line_detect_r2: now also U7.11 (P6)
- net line_detect_r3: now also U7.12 (P7)
- net enable_tof4: no longer names the net of U21.3 (enable_next_board_3v3)
- new net: R12.1, U7.3 (A2)
- new net: R10.1, U7.1 (A0)
- new net: R11.1, U7.2 (A1)
- new net i2C_io_int_3v3: R9.2, U7.13 (~{INT})
- new net scl_3v3: U7.14 (SCL)
- new net sda_3v3: U7.15 (SDA)
Other:
- moved on the sheet: R32, R33, U10, U17, U21, U6
