File: elec/hw/cartes/pmi_2023/power_supply.kicad_sch (KiCad schematic)
At the start: 0 parts

Commit message: pmi2023 wip
Parts:
- added C47: 1µF 16V, symbol cocotter_capacitors:C_1µF_16V_0805
- added C48: 10µF 16V, symbol cocotter_capacitors:C_10µF_16V_0805
- added R10, R11: 0R, cocotter_resistor:r0603_reflow, symbol cocotter_resistors:R_0R_0603
- added U34: ~, symbol cocotter_ic:ST1S03PUR
- added U35: ST1S41PHR, symbol cocotter_ic:ST1S41PHR
Connections:
- new net: C47.1, R10.1, R11.2, U35.1 (Vin_ana)
- new net: R10.2, U35.2 (EN)
- new net +BATT: C48.1, R11.1, U35.7 (Vin_sw)
- new net GND: C47.2, C48.2, U35.4 (GND), U35.8 (PGND), U35.EP (GND)
Other:
- note added: "ajout lm74720"

Commit message: pmi_2023 wip
Parts:
- added J4: ~, cocotter_connectors:1051, symbol cocotter_connectors:1051
- C47, C48: footprint (none) -> cocotter_capacitors:C_0805_2012Metric
Connections:
- net +BATT: now also J4.+
- net GND: now also J4.-
Other:
- note added: "tlv61070a"
- note added: "utiliser bq25173"
Changed lines of the file:
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@@
+    (stroke (width 0) (type default))
+  )
+  (wire (pts (xy 26.67 54.61) (xy 26.67 57.15))
     (stroke (width 0) (type default))
   )
@@
     (stroke (width 0) (type default))
   )
+  (wire (pts (xy 26.67 67.31) (xy 26.67 69.85))
+    (stroke (width 0) (type default))
+  )
   (wire (pts (xy 63.5 58.42) (xy 67.31 58.42))
     (stroke (width 0) (type default))
@@
     (stroke (width 0) (type default))
   )
+  (text "utiliser bq25173" (at 30.48 24.13 0)
+    (effects (font (size 1.27 1.27)) (justify left bottom))
+  )
   (text "ajout lm74720" (at 43.18 97.79 0)
+    (effects (font (size 1.27 1.27)) (justify left bottom))
+  )
+  (text "tlv61070a\n" (at 49.53 118.11 0)
     (effects (font (size 1.27 1.27)) (justify left bottom))
   )
@@
     )
   )
+  (symbol (lib_id "cocotter_connectors:1051") (at 26.67 62.23 0) (unit 1)
+    (in_bom yes) (on_board yes) (dnp no) (fields_autoplaced)
+    (property "Reference" "J4" (at 35.56 63.0583 0)
+      (effects (font (size 1.27 1.27)) (justify left))
+    )
+    (property "Value" "~" (at 26.67 62.23 0)
+      (effects (font (size 1.27 1.27)))
+    )
+    (property "Footprint" "cocotter_connectors:1051" (at 26.67 62.23 0)
+      (effects (font (size 1.27 1.27)) hide)
+    )
+    (property "Datasheet" "https://www.mouser.fr/datasheet/2/215/1051-1112849.pdf" (at 26.67 62.23 0)
+      (effects (font (size 1.27 1.27)) hide)
+    )
+    (pin "+")
+    (pin "-")
+    (instances
+      (project "pmi_2023"
+        (path "/334a657f-c66c-4260-9567-14f1c99913d7/5ea42701-5087-46e6-be28-1d7732af67f5"
+          (reference "J4") (unit 1)
+        )
+      )
+    )
+  )
   (symbol (lib_id "cocotter_resistors:R_0R_0603") (at 73.66 60.96 90) (unit 1)
     (in_bom yes) (on_board yes) (dnp no)
@@
     )
   )
+  (symbol (lib_id "power:+BATT") (at 26.67 54.61 0) (unit 1)
+    (in_bom yes) (on_board yes) (dnp no) (fields_autoplaced)
+    (property "Reference" "#PWR024" (at 26.67 58.42 0)
+      (effects (font (size 1.27 1.27)) hide)
+    )
+    (property "Value" "+BATT" (at 26.67 49.53 0)
+      (effects (font (size 1.27 1.27)))
+    )
+    (property "Footprint" "" (at 26.67 54.61 0)
+      (effects (font (size 1.27 1.27)) hide)
+    )
+    (property "Datasheet" "" (at 26.67 54.61 0)
+      (effects (font (size 1.27 1.27)) hide)
+    )
+    (pin "1")
+    (instances
+      (project "pmi_2023"
+        (path "/334a657f-c66c-4260-9567-14f1c99913d7/5ea42701-5087-46e6-be28-1d7732af67f5"
+          (reference "#PWR024") (unit 1)
+        )
+      )
+    )
+  )
   (symbol (lib_id "power:GND") (at 88.9 69.85 0) (unit 1)
     (in_bom yes) (on_board yes) (dnp no) (fields_autoplaced)
@@
       (effects (font (size 1.27 1.27)) (justify left))
     )
-    (property "Footprint" "" (at 64.4652 69.85 0)
+    (property "Footprint" "cocotter_capacitors:C_0805_2012Metric" (at 64.4652 69.85 0)
       (effects (font (size 1.27 1.27)) hide)
     )
@@
       (effects (font (size 1.27 1.27)) (justify left))
     )
-    (property "Footprint" "" (at 46.6852 69.85 0)
+    (property "Footprint" "cocotter_capacitors:C_0805_2012Metric" (at 46.6852 69.85 0)
       (effects (font (size 1.27 1.27)) hide)
     )
@@
         )
       )
+    )
+  )
+  (symbol (lib_id "power:GND") (at 26.67 69.85 0) (unit 1)
+    (in_bom yes) (on_board yes) (dnp no) (fields_autoplaced)
+    (property "Reference" "#PWR012" (at 26.67 76.2 0)
+      (effects (font (size 1.27 1.27)) hide)
+    )
+    (property "Value" "GND" (at 26.67 74.93 0)
+      (effects (font (size 1.27 1.27)))
+    )
+    (property "Footprint" "" (at 26.67 69.85 0)
+      (effects (font (size 1.27 1.27)) hide)
+    )
+    (property "Datasheet" "" (at 26.67 69.85 0)
+      (effects (font (size 1.27 1.27)) hide)
+    )
+    (pin "1")
+    (instances
+      (project "pmi_2023"
+        (path "/334a657f-c66c-4260-9567-14f1c99913d7/5ea42701-5087-46e6-be28-1d7732af67f5"
+          (reference "#PWR012") (unit 1)
+        )
+      )

Commit message: wip
Parts:
- removed C47: 1µF 16V, cocotter_capacitors:C_0805_2012Metric, symbol cocotter_capacitors:C_1µF_16V_0805
- removed C48: 10µF 16V, cocotter_capacitors:C_0805_2012Metric, symbol cocotter_capacitors:C_10µF_16V_0805
- removed J4: ~, cocotter_connectors:1051, symbol cocotter_connectors:1051
- removed R10, R11: 0R, cocotter_resistor:r0603_reflow, symbol cocotter_resistors:R_0R_0603
- removed U34: ~, symbol cocotter_ic:ST1S03PUR
- removed U35: ST1S41PHR, symbol cocotter_ic:ST1S41PHR
- added BT1: Battery_Cell, symbol Device:Battery_Cell
- added C27, C30, C39, C40: 10µF 16V, cocotter_capacitors:C_0805_2012Metric, symbol cocotter_capacitors:C_10µF_16V_0805
- added C29, C37, C41, C42: 18nF 50V, cocotter_capacitors:C_0603_1608Metric, symbol cocotter_capacitors:C_18nF_50V_0603
- added C36, C38, C43, C44: 47µF 10V, cocotter_capacitors:C_1206_3216Metric, symbol cocotter_capacitors:C_47µF_10V_1206_X5R
- added C45: 1µF 50V, cocotter_capacitors:C_0805_2012Metric, symbol cocotter_capacitors:C_1µF_50V_0805
- added C46: 10µF 25V, cocotter_capacitors:C_0805_2012Metric, symbol cocotter_capacitors:C_10µF_16V_0805_X5R
- added D7: red, 0603, cocotter_diodes:LED_0603_1608Metric, symbol cocotter_diodes:white_led_0603
- added F1: fuse_holder_5x20mm_TH, cocotter_connectors:PTF-15, symbol cocotter_connectors:fuse_holder_5x20mm_TH
- added J5, J8: 254, cocotter_connectors:MY-18650-02, symbol cocotter_connectors:254
- added L1, L2, L3, L4: 2.2µH, cocotter_inductors:L_Kyocera_07A7_7.3x6.6mm, symbol cocotter_inductors:LMLP07A7M2R2DTAS
- added Q3: DMP2008UFG-7, cocotter_transistors:Diodes_PowerDI3333-8, symbol cocotter_transistors:DMP2008UFG-7
- added R103, R104, R105, R106, R65: 0R, cocotter_resistor:r0603_reflow, symbol cocotter_resistors:R_0R_0603
- added R107, R108, R111, R113: 10k, cocotter_resistor:r0603_reflow, symbol cocotter_resistors:R_10k_0603_1%
- added R110, R112, R67: 90k, cocotter_resistor:r0603_reflow, symbol cocotter_resistors:R_90k_0603_1%
- added R114: 1k 1%, cocotter_resistor:r0603_reflow, symbol cocotter_resistors:R_1k_0603_1%
- added R66: 68k 1%, cocotter_resistor:r0603_reflow, symbol cocotter_resistors:R_68k_0603_1%
- added SW8: MSS12C02LS-BB2.0, cocotter_connectors:MSS12C02LS-BB2.0, symbol cocotter_connectors:MSS12C02LS-BB2.0
- added U28, U29, U33, U34: TLV61070A, cocotter_ic:SOT-23-6, symbol cocotter_ic:TLV61070A
- added U35: LDL1117S33R, cocotter_ic:SOT-223, symbol cocotter_ic:LDL1117S33R
Connections:
- net +5V: now also C37.1, C38.1, R67.1, U29.5 (Vout)
- net +BATT: now also C27.1, C30.1, C39.1, C40.1, F1.1, L1.1, L2.1, L3.1, L4.1, R103.2, R104.2, R105.2, R106.2, R114.1, R65.1, U28.6 (Vin), U29.6 (Vin), U33.6 (Vin), U34.6 (Vin)
- net GND: now also C27.2, C30.2, C36.2, C38.2, C39.2, C40.2, C43.2, C44.2, C45.2, C46.2, D7.C, J5.1, Q3.4 (G), R107.2, R108.2, R111.2, R113.2, SW8.B, U28.2 (GND), U29.2 (GND), U33.2 (GND), U34.2 (GND), U35.1 (GND)
- new net: L3.2, U33.1 (SW)
- new net: C41.2, R110.2, R111.1, U33.4 (FB)
- new net: F1.2, Q3.1 (S), Q3.2 (S), Q3.3 (S), R103.1, R104.1, R105.1, R106.1
- new net: J8.1, Q3.5 (D)
- new net: C29.2, R107.1, R66.2, U28.4 (FB)
- new net: C37.2, R108.1, R67.2, U29.4 (FB)
- new net: L1.2, U28.1 (SW)
- new net: C42.2, R112.2, R113.1, U34.4 (FB)
- new net: L4.2, U34.1 (SW)
- new net: L2.2, U29.1 (SW)
- new net +3.3V: C46.1, U35.2 (Vout), U35.4 (Vout)
- new net P3V9: C29.1, C36.1, C45.1, R66.1, U28.5 (Vout), U35.3 (Vin)
- new net Vmot_left_5V: C41.1, C43.1, R110.1, U33.5 (Vout)
- new net Vmot_right_5V: C42.1, C44.1, R112.1, U34.5 (Vout)
- new net enable_pw_conv_3v7: D7.A, R114.2, SW8.A, U28.3 (EN), U29.3 (EN), U33.3 (EN), U34.3 (EN)
- new net vbatt_mon_4.35V: R65.2
Other:
- note added: "0.3A"
- note added: "0.4A"
- note added: "0.5A"
- note added: "0.6A"
- note added: "1.3A"
- note added: "2.1A"
- note added: "2.3A"
- note added: "7.0A"
- note added: "730mA"
- note added: "POWER TREE"
- note added: "boost : TLV61070A"
- note added: "passer en 18650, 1800mAh https://fr.aliexpress.com/item/1005005364329204.html?spm=a2g0o.productlist.main.1.79e32430zv9uBR&algo_pvid=b51d1612-023c-4deb-90a4-82b642b6877c&algo_exp_id=b51d1612-023c-4deb-90a4-82b642b6877c-0&pdp_npi=4%40dis%21EUR%2132.58%2120.2%21%21%2135.26%21%21%40211b813c17039785284962835e8012%2112000032749290547%21sea%21FR%210%21AB&curPageLogUid=3OSaMYC8x88B"
- note added: "use 10A fuses"

Commit message: wip
Parts:
- removed F1: fuse_holder_5x20mm_TH, cocotter_connectors:PTF-15, symbol cocotter_connectors:fuse_holder_5x20mm_TH
- added F1, F2, F3: 10A F, cocotter_others:JFC2410, symbol cocotter_others:JFC2410-2100FS
- R114: Specification 10k 0603 1% 100mW -> 1k 0603 1% 100mW
Connections:
- net +BATT: now also F1.2
- net at Q3.1 (S), Q3.2 (S), Q3.3 (S)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: now also F1.1
Other:
- note added: "SPARE FUSES"
- note removed: "use 10A fuses"
Changed lines of the file:
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@@
     (stroke (width 0) (type default))
   )
+  (wire (pts (xy 22.86 16.51) (xy 22.86 34.29))
+    (stroke (width 0) (type default))
+  )
   (wire (pts (xy 52.07 31.75) (xy 52.07 36.83))
     (stroke (width 0) (type default))
@@
     (stroke (width 0) (type default))
   )
+  (wire (pts (xy 22.86 16.51) (xy 39.37 16.51))
+    (stroke (width 0) (type default))
+  )
   (wire (pts (xy 234.95 160.02) (xy 260.35 160.02))
     (stroke (width 0) (type default))
@@
     (stroke (width 0) (type default))
   )
+  (wire (pts (xy 39.37 34.29) (xy 39.37 16.51))
+    (stroke (width 0) (type default))
+  )
   (wire (pts (xy 59.69 31.75) (xy 59.69 36.83))
     (stroke (width 0) (type default))
@@
     (stroke (width 0) (type default))
   )
+  (wire (pts (xy 22.86 34.29) (xy 39.37 34.29))
+    (stroke (width 0) (type default))
+  )
   (wire (pts (xy 262.89 30.48) (xy 262.89 27.94))
     (stroke (width 0) (type default))
@@
     (effects (font (size 1.27 1.27) bold) (justify left bottom))
   )
+  (text "SPARE FUSES" (at 24.13 19.05 0)
+    (effects (font (size 1.27 1.27) (thickness 0.254) bold) (justify left bottom))
+  )
   (text "7.0A" (at 41.91 127 0)
     (effects (font (size 1.27 1.27)) (justify left bottom))
@@
     (effects (font (size 1.27 1.27)) (justify left bottom))
   )
-  (text "use 10A fuses" (at 52.07 21.59 0)
-    (effects (font (size 1.27 1.27)) (justify left bottom))
-  )
   (text "730mA" (at 114.3 116.84 0)
     (effects (font (size 1.27 1.27)) (justify left bottom))
@@
     )
   )
+  (symbol (lib_id "cocotter_others:JFC2410-2100FS") (at 55.88 26.67 0) (unit 1)
+    (in_bom yes) (on_board yes) (dnp no)
+    (property "Reference" "F1" (at 55.88 25.4 0)
+      (effects (font (size 1.27 1.27)))
+    )
+    (property "Value" "10A F" (at 63.5 26.67 0)
+      (effects (font (size 1.27 1.27)))
+    )
+    (property "Footprint" "cocotter_others:JFC2410" (at 55.88 26.67 0)
+      (effects (font (size 1.27 1.27)) hide)
+    )
+    (property "Datasheet" "https://datasheet.lcsc.com/lcsc/2305151203_Shenzhen-JDT-Fuse-JFC2410-2100FS_C136374.pdf" (at 55.88 29.21 0)
+      (effects (font (size 1.27 1.27)) hide)
+    )
+    (property "JLCPCB" "C136374" (at 55.88 29.21 0)
+      (effects (font (size 1.27 1.27)) hide)
+    )
+    (pin "1")
+    (pin "2")
+    (instances
+      (project "pmi_2023"
+        (path "/334a657f-c66c-4260-9567-14f1c99913d7/5ea42701-5087-46e6-be28-1d7732af67f5"
+          (reference "F1") (unit 1)
+        )
+      )
+    )
+  )
   (symbol (lib_id "cocotter_inductors:LMLP07A7M2R2DTAS") (at 222.25 95.25 90) (unit 1)
     (in_bom yes) (on_board yes) (dnp no) (fields_autoplaced)
@@
     )
   )
+  (symbol (lib_id "cocotter_others:JFC2410-2100FS") (at 29.21 22.86 0) (unit 1)
+    (in_bom yes) (on_board yes) (dnp no)
+    (property "Reference" "F2" (at 29.21 20.32 0)
+      (effects (font (size 1.27 1.27)))
+    )
+    (property "Value" "10A F" (at 29.21 25.4 0)
+      (effects (font (size 1.27 1.27)))
+    )
+    (property "Footprint" "cocotter_others:JFC2410" (at 29.21 22.86 0)
+      (effects (font (size 1.27 1.27)) hide)
+    )
+    (property "Datasheet" "https://datasheet.lcsc.com/lcsc/2305151203_Shenzhen-JDT-Fuse-JFC2410-2100FS_C136374.pdf" (at 29.21 25.4 0)
+      (effects (font (size 1.27 1.27)) hide)
+    )
+    (property "JLCPCB" "C136374" (at 29.21 25.4 0)
+      (effects (font (size 1.27 1.27)) hide)
+    )
+    (pin "2")
+    (pin "1")
+    (instances
+      (project "pmi_2023"
+        (path "/334a657f-c66c-4260-9567-14f1c99913d7/5ea42701-5087-46e6-be28-1d7732af67f5"
+          (reference "F2") (unit 1)
+        )
+      )
+    )
+  )
   (symbol (lib_id "power:+BATT") (at 67.31 39.37 0) (unit 1)
     (in_bom yes) (on_board yes) (dnp no) (fields_autoplaced)
@@
     )
   )
+  (symbol (lib_id "cocotter_others:JFC2410-2100FS") (at 29.21 30.48 0) (unit 1)
+    (in_bom yes) (on_board yes) (dnp no)
+    (property "Reference" "F3" (at 29.21 27.94 0)
+      (effects (font (size 1.27 1.27)))
+    )
+    (property "Value" "10A F" (at 29.21 33.02 0)
+      (effects (font (size 1.27 1.27)))
+    )
+    (property "Footprint" "cocotter_others:JFC2410" (at 29.21 30.48 0)
+      (effects (font (size 1.27 1.27)) hide)
+    )
+    (property "Datasheet" "https://datasheet.lcsc.com/lcsc/2305151203_Shenzhen-JDT-Fuse-JFC2410-2100FS_C136374.pdf" (at 29.21 33.02 0)
+      (effects (font (size 1.27 1.27)) hide)
+    )
+    (property "JLCPCB" "C136374" (at 29.21 33.02 0)
+      (effects (font (size 1.27 1.27)) hide)
+    )
+    (pin "2")
+    (pin "1")
+    (instances
+      (project "pmi_2023"
+        (path "/334a657f-c66c-4260-9567-14f1c99913d7/5ea42701-5087-46e6-be28-1d7732af67f5"
+          (reference "F3") (unit 1)
+        )
+      )
+    )
+  )
   (symbol (lib_id "power:GND") (at 29.21 69.85 0) (unit 1)
     (in_bom yes) (on_board yes) (dnp no) (fields_autoplaced)
@@
     )
   )
-  (symbol (lib_id "cocotter_connectors:fuse_holder_5x20mm_TH") (at 55.88 26.67 0) (unit 1)
-    (in_bom yes) (on_board yes) (dnp no) (fields_autoplaced)
-    (property "Reference" "F1" (at 55.88 24.13 0)
-      (effects (font (size 1.27 1.27)))
-    )
-    (property "Value" "fuse_holder_5x20mm_TH" (at 53.975 26.67 0)
-      (effects (font (size 1.27 1.27)) hide)
-    )
-    (property "Footprint" "cocotter_connectors:PTF-15" (at 55.88 24.892 0)
-      (effects (font (size 1.27 1.27)) hide)
-    )
-    (property "Datasheet" "https://datasheet.lcsc.com/lcsc/2011091603_Xucheng-Elec-C58066_C58066.pdf" (at 55.88 26.67 90)
-      (effects (font (size 1.27 1.27)) hide)
-    )
-    (property "JLCPCB" "C58066" (at 55.88 26.67 0)
-      (effects (font (size 1.27 1.27)) hide)
-    )
-    (pin "1")
-    (pin "2")
-    (instances
-      (project "pmi_2023"
-        (path "/334a657f-c66c-4260-9567-14f1c99913d7/5ea42701-5087-46e6-be28-1d7732af67f5"
-          (reference "F1") (unit 1)
-        )
-      )
-    )
-  )
   (symbol (lib_id "cocotter_resistors:R_0R_0603") (at 55.88 41.91 90) (unit 1)
     (in_bom yes) (on_board yes) (dnp yes)
@@
       (effects (font (size 1.27 1.27)) hide)
     )
-    (property "Specification" "10k 0603 1% 100mW" (at 59.69 52.07 0)
+    (property "Specification" "1k 0603 1% 100mW" (at 59.69 52.07 0)
       (effects (font (size 1.27 1.27)) hide)
     )
