File: elec/hw/cartes/pmi_2023/propulsion.kicad_sch (KiCad schematic)
At the start: 55 parts, among them U1 DRV8231ADDAR, U2 SN74LVC1T45DBV, U3 SN74LVC1T45DBV, U4 DRV8231ADDAR, U5 SN74LVC1T45DBV, U6 SN74LVC1T45DBV, U7 SN74LVC1T45DBV

Commit message: pmi2023 wip
Parts:
- removed R10, R11, R19, R20, R21, R22: 0R, cocotter_resistor:r0603_reflow, symbol cocotter_resistors:R_0R_0603
- added C40, C41: 100nF 50V, symbol cocotter_capacitors:C_100nF_50V_0603
- added C43: 10µF 16V, symbol cocotter_capacitors:C_10µF_16V_0805
- added J3: con_servo, symbol cocotter_connectors:con_servo
- added ML, MR: motor-JGA12-N20, symbol cocotter_connectors:motor-JGA12-N20
- R32, R7: now not fitted
Connections:
- net GND: now also C40.2, C41.2, C43.2, J3.1 (GND), ML.6 (GND), MR.6 (GND)
- net left_encod_A_5V: now also ML.3 (HALL_A)
- net left_encod_B_5V: now also ML.4 (HALL_B)
- net pwm_vaccum_5v: now also J3.3 (PWM)
- net right_encod_A_5V: now also MR.3 (HALL_A)
- net right_encod_B_5V: now also MR.4 (HALL_B)
- net encoder_supply: now reaches C14.1, U6.6 (VCCB)
- net encoder_supply: now also C13.1, C6.1, C7.1, R6.2, R7.2, U2.6 (VCCB), U3.6 (VCCB), U5.6 (VCCB), C40.1, C41.1, ML.5 (5V), MR.5 (5V)
- net at C18.1, R31.1, R32.1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: now also C43.1, J3.2 (5V)
- net at U1.6 (OUT1): now also ML.1 (M+)
- net at U1.8 (OUT2): now also ML.2 (M-)
- net at U4.6 (OUT1): now also MR.1 (M+)
- net at U4.8 (OUT2): now also MR.2 (M-)
Other:
- note removed: "manque connecteur regulateur"
- note removed: "manque symbole pour moteur + codeur"
- moved on the sheet: C18, R31

Commit message: pmi_2023 wip
Parts:
- removed R13, R25, R26: 0R, cocotter_resistor:r0603_reflow, symbol cocotter_resistors:R_0R_0603
- added R19: 100k, cocotter_resistor:r0603_reflow, symbol cocotter_resistors:R_100k_0603_1%
- C1, C10, C13, C14, C15, C16, C17, C18, C2, C40, C41, C5, C6, C7, C8, C9: footprint (none) -> cocotter_capacitors:C_0603_1608Metric
- C11, C12, C3, C4: footprint (none) -> cocotter_capacitors:C_1206_3216Metric
- C43: footprint (none) -> cocotter_capacitors:C_0805_2012Metric
- J3: footprint (none) -> cocotter_connectors:ana_servo_5V
- U1, U4: footprint (none) -> cocotter_ic:DDA0008B
- renumbered ML to ML1, MR to MR1
Connections:
- net +3.3V: now also R19.1
- net GND: now also U1.9 (PAD), U4.9 (PAD)
- net nREAD_encoder_3v3: now reaches U6.5 (DIR)
- net nREAD_encoder_3v3: now also R9.2, U2.5 (DIR), U3.5 (DIR), U5.5 (DIR), R19.2
Other:
- note added: "9 signaux controle"
- note added: "pilotage du moteur par pwm et mos ref jlcpcb C2938374 remplacement translateurs niveau par eesx1321"

Commit message: wip
Parts:
- removed C12, C4: 22µF 16V, cocotter_capacitors:C_1206_3216Metric, symbol cocotter_capacitors:C_22µF_16V_1206_X5R
- removed C13, C15, C16, C17, C18, C40, C41, C5, C6, C7: 100nF 50V, cocotter_capacitors:C_0603_1608Metric, symbol cocotter_capacitors:C_100nF_50V_0603
- removed C43: 10µF 16V, cocotter_capacitors:C_0805_2012Metric, symbol cocotter_capacitors:C_10µF_16V_0805
- removed J3: con_servo, cocotter_connectors:ana_servo_5V, symbol cocotter_connectors:con_servo
- removed ML1, MR1: motor-JGA12-N20, symbol cocotter_connectors:motor-JGA12-N20
- removed R12, R19, R23, R24, R8: 100k, cocotter_resistor:r0603_reflow, symbol cocotter_resistors:R_100k_0603_1%
- removed R16, R17, R3, R4: 10k, cocotter_resistor:r0603_reflow, symbol cocotter_resistors:R_10k_0603_1%
- removed R32, R6, R7, R9: 0R, cocotter_resistor:r0603_reflow, symbol cocotter_resistors:R_0R_0603
- removed U2, U3, U5, U6, U7: SN74LVC1T45DBV, Package_TO_SOT_SMD:SOT-23-6, symbol cocotter_ic:SN74LVC1T45DBV
- added Q1: ~, cocotter_transistors:SOT-23-3, symbol cocotter_transistors:SI2310
- added R13, R14, R15, R16, R17, R18, R19, R20, R21, R22, R23, R24, R25, R26, R27, R28: 1k 1%, cocotter_resistor:r0603_reflow, symbol cocotter_resistors:R_1k_0603_1%
- added R29: 0R, cocotter_resistor:r0603_reflow, symbol cocotter_resistors:R_0R_0603
- added TP1, TP2, TP3, TP4, TP5, TP6: TestPoint, cocotter_others:testpoint-THT-0.5mm, symbol cocotter_others:TestPoint
- added U3, U4: EESX1321, cocotter_ic:EESX1321, symbol cocotter_ic:EESX1321
- C1, C8: JLCPCB (none) -> C14663
- C2: renamed from C9; JLCPCB (none) -> C14663
- C3: renamed from C2; JLCPCB (none) -> C14663
- C4: renamed from C10; JLCPCB (none) -> C14663
- C5: renamed from C3; value 22µF 16V -> 47µF 10V; symbol cocotter_capacitors:C_22µF_16V_1206_X5R -> cocotter_capacitors:C_47µF_10V_1206_X5R; JLCPCB (none) -> C96123; Specification 10µF 16V X7R 0805 -> 47µF 10V X5R 1206
- C6: renamed from C11; value 22µF 16V -> 47µF 10V; symbol cocotter_capacitors:C_22µF_16V_1206_X5R -> cocotter_capacitors:C_47µF_10V_1206_X5R; JLCPCB (none) -> C96123; Specification 10µF 16V X7R 0805 -> 47µF 10V X5R 1206
- C7: renamed from C14; JLCPCB (none) -> C14663
- R1: renamed from R2; JLCPCB (none) -> C25803
- R2: renamed from R14; JLCPCB (none) -> C25803
- R3: renamed from R1; JLCPCB (none) -> C25803
- R30: JLCPCB (none) -> C21189; now not fitted
- R4: renamed from R15; JLCPCB (none) -> C25803
- R5: renamed from R29; JLCPCB (none) -> C25803
- R6: renamed from R18; value 10k -> 3k3 1%; symbol cocotter_resistors:R_10k_0603_1% -> cocotter_resistors:R_3k3_0603_1%; Specification 10k 0603 1% 100mW -> 3k3 0603 1% 100mW; mouser 603-RC0603FR-10100KL -> (none)
- R7: renamed from R5; value 10k -> 3k3 1%; symbol cocotter_resistors:R_10k_0603_1% -> cocotter_resistors:R_3k3_0603_1%; Specification 10k 0603 1% 100mW -> 3k3 0603 1% 100mW; mouser 603-RC0603FR-10100KL -> (none)
- R8: renamed from R31; JLCPCB (none) -> C21189
- U1: JLCPCB (none) -> C5218849
- U2: renamed from U4; JLCPCB (none) -> C5218849
Connections:
- net +3.3V: now also U3.1 (A), U4.1 (A); no longer C8.1
- net +5V: now also R29.2; no longer R8.2
- net GND: now also Q1.2 (S), R13.2, R14.2, R15.2, R16.2, R18.2, R21.2, R23.2, R27.2
- net encoder_supply: now also C8.1, R30.1, R29.1, U3.6 (C), U4.6 (C)
- net left_encod_A_3v3: now also R26.2, R27.1, R28.2
- net left_encod_B_3v3: now also R20.2, R21.1, R24.2
- net pwm_vaccum_3v3: now also Q1.1 (G)
- net right_encod_A_3v3: now also R22.2, R23.1, R25.2
- net right_encod_B_3v3: now also R17.2, R18.1, R19.2
- net at R8.1: now also TP1.1
- net mot_right_A: now reaches U2.6 (OUT1)
- net mot_right_A: now also TP5.1
- net mot_right_B: now reaches U2.8 (OUT2)
- net mot_right_B: now also TP6.1
- net mot_left_A: now reaches U1.6 (OUT1)
- net mot_left_A: now also TP3.1
- net mot_left_B: now reaches U1.8 (OUT2)
- net mot_left_B: now also TP4.1
- net +BATT renamed Vmot_left_5V
- net Vmot_left_5V: now also R8.2; no longer C4.1, C6.1, U2.5 (VM)
- new net: R14.1, U3.3 (C2)
- new net: R22.1, R25.1, U3.4 (E1)
- new net: R17.1, R19.1, U3.5 (E2)
- new net: R26.1, R28.1, U4.4 (E1)
- new net: Q1.3 (D), TP2.1
- new net: R20.1, R24.1, U4.5 (E2)
- new net: R13.1, U3.2 (C1)
- new net: R15.1, U4.2 (C1)
- new net: R16.1, U4.3 (C2)
- new net Vmot_right_5V: C4.1, C6.1, U2.5 (VM)
Other:
- note added: "utiliser res 3k3"
- moved on the sheet: C7, R6, R7, R8

Commit message: wip
Parts:
- R13, R14, R15, R16, R17, R18, R19, R20, R21, R22, R23, R24, R25, R26, R27, R28: Specification 10k 0603 1% 100mW -> 1k 0603 1% 100mW
Changed lines of the file:
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@@
       (effects (font (size 1.27 1.27)) hide)
     )
-    (property "Specification" "10k 0603 1% 100mW" (at 171.45 135.89 0)
+    (property "Specification" "1k 0603 1% 100mW" (at 171.45 135.89 0)
       (effects (font (size 1.27 1.27)) hide)
     )
@@
       (effects (font (size 1.27 1.27)) hide)
     )
-    (property "Specification" "10k 0603 1% 100mW" (at 218.44 123.19 0)
+    (property "Specification" "1k 0603 1% 100mW" (at 218.44 123.19 0)
       (effects (font (size 1.27 1.27)) hide)
     )
@@
       (effects (font (size 1.27 1.27)) hide)
     )
-    (property "Specification" "10k 0603 1% 100mW" (at 187.96 127 0)
+    (property "Specification" "1k 0603 1% 100mW" (at 187.96 127 0)
       (effects (font (size 1.27 1.27)) hide)
     )
@@
       (effects (font (size 1.27 1.27)) hide)
     )
-    (property "Specification" "10k 0603 1% 100mW" (at 198.12 127 0)
+    (property "Specification" "1k 0603 1% 100mW" (at 198.12 127 0)
       (effects (font (size 1.27 1.27)) hide)
     )
@@
       (effects (font (size 1.27 1.27)) hide)
     )
-    (property "Specification" "10k 0603 1% 100mW" (at 219.71 45.72 0)
+    (property "Specification" "1k 0603 1% 100mW" (at 219.71 45.72 0)
       (effects (font (size 1.27 1.27)) hide)
     )
@@
       (effects (font (size 1.27 1.27)) hide)
     )
-    (property "Specification" "10k 0603 1% 100mW" (at 199.39 49.53 0)
+    (property "Specification" "1k 0603 1% 100mW" (at 199.39 49.53 0)
       (effects (font (size 1.27 1.27)) hide)
     )
@@
       (effects (font (size 1.27 1.27)) hide)
     )
-    (property "Specification" "10k 0603 1% 100mW" (at 209.55 49.53 0)
+    (property "Specification" "1k 0603 1% 100mW" (at 209.55 49.53 0)
       (effects (font (size 1.27 1.27)) hide)
     )
@@
       (effects (font (size 1.27 1.27)) hide)
     )
-    (property "Specification" "10k 0603 1% 100mW" (at 219.71 58.42 0)
+    (property "Specification" "1k 0603 1% 100mW" (at 219.71 58.42 0)
       (effects (font (size 1.27 1.27)) hide)
     )
@@
       (effects (font (size 1.27 1.27)) hide)
     )
-    (property "Specification" "10k 0603 1% 100mW" (at 208.28 135.89 0)
+    (property "Specification" "1k 0603 1% 100mW" (at 208.28 135.89 0)
       (effects (font (size 1.27 1.27)) hide)
     )
@@
       (effects (font (size 1.27 1.27)) hide)
     )
-    (property "Specification" "10k 0603 1% 100mW" (at 229.87 45.72 0)
+    (property "Specification" "1k 0603 1% 100mW" (at 229.87 45.72 0)
       (effects (font (size 1.27 1.27)) hide)
     )
@@
       (effects (font (size 1.27 1.27)) hide)
     )
-    (property "Specification" "10k 0603 1% 100mW" (at 161.29 135.89 0)
+    (property "Specification" "1k 0603 1% 100mW" (at 161.29 135.89 0)
       (effects (font (size 1.27 1.27)) hide)
     )
@@
       (effects (font (size 1.27 1.27)) hide)
     )
-    (property "Specification" "10k 0603 1% 100mW" (at 208.28 123.19 0)
+    (property "Specification" "1k 0603 1% 100mW" (at 208.28 123.19 0)
       (effects (font (size 1.27 1.27)) hide)
     )
@@
       (effects (font (size 1.27 1.27)) hide)
     )
-    (property "Specification" "10k 0603 1% 100mW" (at 182.88 58.42 0)
+    (property "Specification" "1k 0603 1% 100mW" (at 182.88 58.42 0)
       (effects (font (size 1.27 1.27)) hide)
     )
@@
       (effects (font (size 1.27 1.27)) hide)
     )
-    (property "Specification" "10k 0603 1% 100mW" (at 187.96 135.89 0)
+    (property "Specification" "1k 0603 1% 100mW" (at 187.96 135.89 0)
       (effects (font (size 1.27 1.27)) hide)
     )
@@
       (effects (font (size 1.27 1.27)) hide)
     )
-    (property "Specification" "10k 0603 1% 100mW" (at 199.39 58.42 0)
+    (property "Specification" "1k 0603 1% 100mW" (at 199.39 58.42 0)
       (effects (font (size 1.27 1.27)) hide)
     )
@@
       (effects (font (size 1.27 1.27)) hide)
     )
-    (property "Specification" "10k 0603 1% 100mW" (at 172.72 58.42 0)
-      (effects (font (size 1.27 1.27)) hide)
-    )
+    (property "Specification" "1k 0603 1% 100mW" (at 172.72 58.42 0)
+      (effects (font (size 1.27 1.27)) hide)
+    )

Commit message: pmi layout (WIP)
Connections:
- net +3.3V renamed +3V3
Changed lines of the file:
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@@
   (junction (at 45.72 118.11) (diameter 0) (color 0 0 0 0)
   )
+  (junction (at 55.88 49.53) (diameter 0) (color 0 0 0 0)
+  )
   (junction (at 81.28 128.27) (diameter 0) (color 0 0 0 0)
   )
@@
   (junction (at 193.04 105.41) (diameter 0) (color 0 0 0 0)
   )
+  (junction (at 209.55 53.34) (diameter 0) (color 0 0 0 0)
+  )
+  (junction (at 104.14 100.33) (diameter 0) (color 0 0 0 0)
+  )
+  (junction (at 121.92 110.49) (diameter 0) (color 0 0 0 0)
+  )
+  (junction (at 52.07 177.8) (diameter 0) (color 0 0 0 0)
+  )
+  (junction (at 219.71 49.53) (diameter 0) (color 0 0 0 0)
+  )
   (junction (at 55.88 125.73) (diameter 0) (color 0 0 0 0)
-  )
-  (junction (at 209.55 53.34) (diameter 0) (color 0 0 0 0)
-  )
-  (junction (at 104.14 100.33) (diameter 0) (color 0 0 0 0)
-  )
-  (junction (at 121.92 110.49) (diameter 0) (color 0 0 0 0)
-  )
-  (junction (at 52.07 177.8) (diameter 0) (color 0 0 0 0)
-  )
-  (junction (at 219.71 49.53) (diameter 0) (color 0 0 0 0)
-  )
-  (junction (at 55.88 49.53) (diameter 0) (color 0 0 0 0)
   )
   (junction (at 218.44 127) (diameter 0) (color 0 0 0 0)
@@
     )
   )
+  (symbol (lib_id "power:+3V3") (at 55.88 125.73 0) (unit 1)
+    (in_bom yes) (on_board yes) (dnp no)
+    (property "Reference" "#PWR026" (at 55.88 129.54 0)
+      (effects (font (size 1.27 1.27)) hide)
+    )
+    (property "Value" "+3V3" (at 55.88 121.92 0)
+      (effects (font (size 1.27 1.27)))
+    )
+    (property "Footprint" "" (at 55.88 125.73 0)
+      (effects (font (size 1.27 1.27)) hide)
+    )
+    (property "Datasheet" "" (at 55.88 125.73 0)
+      (effects (font (size 1.27 1.27)) hide)
+    )
+    (pin "1")
+    (instances
+      (project "pmi_2023"
+        (path "/334a657f-c66c-4260-9567-14f1c99913d7/e27753ab-5deb-4e63-8abb-23778f088204"
+          (reference "#PWR026") (unit 1)
+        )
+      )
+    )
+  )
   (symbol (lib_id "power:GND") (at 82.55 64.77 0) (unit 1)
     (in_bom yes) (on_board yes) (dnp no) (fields_autoplaced)
@@
     )
   )
+  (symbol (lib_id "power:+3V3") (at 55.88 49.53 0) (unit 1)
+    (in_bom yes) (on_board yes) (dnp no)
+    (property "Reference" "#PWR027" (at 55.88 53.34 0)
+      (effects (font (size 1.27 1.27)) hide)
+    )
+    (property "Value" "+3V3" (at 55.88 45.72 0)
+      (effects (font (size 1.27 1.27)))
+    )
+    (property "Footprint" "" (at 55.88 49.53 0)
+      (effects (font (size 1.27 1.27)) hide)
+    )
+    (property "Datasheet" "" (at 55.88 49.53 0)
+      (effects (font (size 1.27 1.27)) hide)
+    )
+    (pin "1")
+    (instances
+      (project "pmi_2023"
+        (path "/334a657f-c66c-4260-9567-14f1c99913d7/e27753ab-5deb-4e63-8abb-23778f088204"
+          (reference "#PWR027") (unit 1)
+        )
+      )
+    )
+  )
   (symbol (lib_id "cocotter_resistors:R_1k_0603_1%") (at 198.12 127 0) (unit 1)
     (in_bom yes) (on_board yes) (dnp no) (fields_autoplaced)
@@
     )
   )
+  (symbol (lib_id "power:+3V3") (at 181.61 39.37 0) (unit 1)
+    (in_bom yes) (on_board yes) (dnp no)
+    (property "Reference" "#PWR028" (at 181.61 43.18 0)
+      (effects (font (size 1.27 1.27)) hide)
+    )
+    (property "Value" "+3V3" (at 181.61 35.56 0)
+      (effects (font (size 1.27 1.27)))
+    )
+    (property "Footprint" "" (at 181.61 39.37 0)
+      (effects (font (size 1.27 1.27)) hide)
+    )
+    (property "Datasheet" "" (at 181.61 39.37 0)
+      (effects (font (size 1.27 1.27)) hide)
+    )
+    (pin "1")
+    (instances
+      (project "pmi_2023"
+        (path "/334a657f-c66c-4260-9567-14f1c99913d7/e27753ab-5deb-4e63-8abb-23778f088204"
+          (reference "#PWR028") (unit 1)
+        )
+      )
+    )
+  )
   (symbol (lib_id "cocotter_resistors:R_100k_0603_1%") (at 52.07 184.15 0) (unit 1)
     (in_bom yes) (on_board yes) (dnp no) (fields_autoplaced)
@@
         (path "/334a657f-c66c-4260-9567-14f1c99913d7/e27753ab-5deb-4e63-8abb-23778f088204"
           (reference "C3") (unit 1)
+        )
+      )
+    )
+  )
+  (symbol (lib_id "power:+3V3") (at 241.3 34.29 0) (unit 1)
+    (in_bom yes) (on_board yes) (dnp no)
+    (property "Reference" "#PWR030" (at 241.3 38.1 0)
+      (effects (font (size 1.27 1.27)) hide)
+    )
+    (property "Value" "+3V3" (at 241.3 30.48 0)
+      (effects (font (size 1.27 1.27)))
+    )
+    (property "Footprint" "" (at 241.3 34.29 0)
+      (effects (font (size 1.27 1.27)) hide)
+    )
+    (property "Datasheet" "" (at 241.3 34.29 0)
+      (effects (font (size 1.27 1.27)) hide)
+    )
+    (pin "1")
+    (instances
+      (project "pmi_2023"
+        (path "/334a657f-c66c-4260-9567-14f1c99913d7/e27753ab-5deb-4e63-8abb-23778f088204"
+          (reference "#PWR030") (unit 1)
         )
       )
@@
     )
   )
-  (symbol (lib_id "power:+3.3V") (at 55.88 49.53 0) (unit 1)
-    (in_bom yes) (on_board yes) (dnp no)
-    (property "Reference" "#PWR0124" (at 55.88 53.34 0)
-      (effects (font (size 1.27 1.27)) hide)
-    )
-    (property "Value" "+3.3V" (at 55.88 45.974 0)
-      (effects (font (size 1.27 1.27)))
-    )
-    (property "Footprint" "" (at 55.88 49.53 0)
-      (effects (font (size 1.27 1.27)) hide)
-    )
-    (property "Datasheet" "" (at 55.88 49.53 0)
-      (effects (font (size 1.27 1.27)) hide)
-    )
-    (pin "1")
-    (instances
-      (project "pmi_2023"
-        (path "/334a657f-c66c-4260-9567-14f1c99913d7/e27753ab-5deb-4e63-8abb-23778f088204"
-          (reference "#PWR0124") (unit 1)
-        )
-      )
-    )
-  )
   (symbol (lib_id "power:GND") (at 182.88 62.23 0) (unit 1)
     (in_bom yes) (on_board yes) (dnp no)
@@
     )
   )
-  (symbol (lib_id "power:+3.3V") (at 170.18 116.84 0) (unit 1)
-    (in_bom yes) (on_board yes) (dnp no)
-    (property "Reference" "#PWR0117" (at 170.18 120.65 0)
-      (effects (font (size 1.27 1.27)) hide)
-    )
-    (property "Value" "+3.3V" (at 170.18 113.284 0)
-      (effects (font (size 1.27 1.27)))
-    )
-    (property "Footprint" "" (at 170.18 116.84 0)
-      (effects (font (size 1.27 1.27)) hide)
-    )
-    (property "Datasheet" "" (at 170.18 116.84 0)
-      (effects (font (size 1.27 1.27)) hide)
-    )
-    (pin "1")
-    (instances
-      (project "pmi_2023"
-        (path "/334a657f-c66c-4260-9567-14f1c99913d7/e27753ab-5deb-4e63-8abb-23778f088204"
-          (reference "#PWR0117") (unit 1)
-        )
-      )
-    )
-  )
   (symbol (lib_id "cocotter_resistors:R_0R_0603") (at 232.41 34.29 90) (unit 1)
     (in_bom yes) (on_board yes) (dnp yes)
@@
     )
   )
-  (symbol (lib_id "power:+3.3V") (at 55.88 125.73 0) (unit 1)
-    (in_bom yes) (on_board yes) (dnp no)
-    (property "Reference" "#PWR0120" (at 55.88 129.54 0)
-      (effects (font (size 1.27 1.27)) hide)
-    )
-    (property "Value" "+3.3V" (at 55.88 122.174 0)
-      (effects (font (size 1.27 1.27)))
-    )
-    (property "Footprint" "" (at 55.88 125.73 0)
-      (effects (font (size 1.27 1.27)) hide)
-    )
-    (property "Datasheet" "" (at 55.88 125.73 0)
-      (effects (font (size 1.27 1.27)) hide)
-    )
-    (pin "1")
-    (instances
-      (project "pmi_2023"
-        (path "/334a657f-c66c-4260-9567-14f1c99913d7/e27753ab-5deb-4e63-8abb-23778f088204"
-          (reference "#PWR0120") (unit 1)
-        )
-      )
-    )
-  )
   (symbol (lib_id "power:GND") (at 81.28 140.97 0) (unit 1)
     (in_bom yes) (on_board yes) (dnp no) (fields_autoplaced)
@@
     )
   )
+  (symbol (lib_id "power:+3V3") (at 170.18 116.84 0) (unit 1)
+    (in_bom yes) (on_board yes) (dnp no)
+    (property "Reference" "#PWR029" (at 170.18 120.65 0)
+      (effects (font (size 1.27 1.27)) hide)
+    )
+    (property "Value" "+3V3" (at 170.18 113.03 0)
+      (effects (font (size 1.27 1.27)))
+    )
+    (property "Footprint" "" (at 170.18 116.84 0)
+      (effects (font (size 1.27 1.27)) hide)
+    )
+    (property "Datasheet" "" (at 170.18 116.84 0)
+      (effects (font (size 1.27 1.27)) hide)
+    )
+    (pin "1")
+    (instances
+      (project "pmi_2023"
+        (path "/334a657f-c66c-4260-9567-14f1c99913d7/e27753ab-5deb-4e63-8abb-23778f088204"
+          (reference "#PWR029") (unit 1)
+        )
+      )
+    )
+  )
   (symbol (lib_id "cocotter_capacitors:C_100nF_50V_0603") (at 193.04 109.22 0) (unit 1)
     (in_bom yes) (on_board yes) (dnp no) (fields_autoplaced)
@@
         (path "/334a657f-c66c-4260-9567-14f1c99913d7/e27753ab-5deb-4e63-8abb-23778f088204"
           (reference "R16") (unit 1)
-        )
-      )
-    )
-  )
-  (symbol (lib_id "power:+3.3V") (at 241.3 34.29 0) (mirror y) (unit 1)
-    (in_bom yes) (on_board yes) (dnp no)
-    (property "Reference" "#PWR0112" (at 241.3 38.1 0)
-      (effects (font (size 1.27 1.27)) hide)
-    )
-    (property "Value" "+3.3V" (at 241.3 30.734 0)
-      (effects (font (size 1.27 1.27)))
-    )
-    (property "Footprint" "" (at 241.3 34.29 0)
-      (effects (font (size 1.27 1.27)) hide)
-    )
-    (property "Datasheet" "" (at 241.3 34.29 0)
-      (effects (font (size 1.27 1.27)) hide)
-    )
-    (pin "1")
-    (instances
-      (project "pmi_2023"
-        (path "/334a657f-c66c-4260-9567-14f1c99913d7/e27753ab-5deb-4e63-8abb-23778f088204"
-          (reference "#PWR0112") (unit 1)
         )
       )
@@
         )
       )
-    )
-  )
-  (symbol (lib_id "power:+3.3V") (at 181.61 39.37 0) (unit 1)
-    (in_bom yes) (on_board yes) (dnp no)
-    (property "Reference" "#PWR0103" (at 181.61 43.18 0)
-      (effects (font (size 1.27 1.27)) hide)
-    )
-    (property "Value" "+3.3V" (at 181.61 35.814 0)
-      (effects (font (size 1.27 1.27)))
-    )
-    (property "Footprint" "" (at 181.61 39.37 0)
-      (effects (font (size 1.27 1.27)) hide)
-    )
-    (property "Datasheet" "" (at 181.61 39.37 0)
-      (effects (font (size 1.27 1.27)) hide)
-    )
-    (pin "1")
-    (instances
-      (project "pmi_2023"
-        (path "/334a657f-c66c-4260-9567-14f1c99913d7/e27753ab-5deb-4e63-8abb-23778f088204"
-          (reference "#PWR0103") (unit 1)
-        )
-      )

Commit message: front and back tof added, selector changed, ready to route
Parts:
- R29, R30, R8: JLCPCB C21189 -> C431718

Commit message: wip
Parts:
- R13, R14, R15, R16, R17, R18, R19, R20, R21, R22, R23, R24, R25, R26, R27, R28: Specification 1k 0603 1% 100mW -> 10k 0603 1% 100mW; mouser (none) -> 603-RC0603FR-10100KL
