File: elec/hw/cartes/pmi_2023/sensor_module.kicad_sch (KiCad schematic)
At the start: 31 parts, among them U22 VL53L5CXV0GC, U27 BMI088, U30 VL53L5CXV0GC

Commit message: pmi: beginning of transition toward 0402 resistors and capacitors, battery gauge added
Parts:
- C12, C20, C53, C57, C58, C59: footprint cocotter_capacitors:C_0603_1608Metric -> cocotter_capacitors:C_0402_1005Metric; symbol cocotter_capacitors:C_100nF_50V_0603 -> cocotter_capacitors:C_100nF_50V_0402; JLCPCB Part # C14663 -> C85858; Specification 100nF 50V X7R 0603 -> 100nF 50V X7R 0402
- R123, R124, R128: footprint cocotter_resistor:r0603_reflow -> cocotter_resistor:r0402_reflow; symbol cocotter_resistors:R_10k_0603_1% -> cocotter_resistors:R_10k_0402_1%; JLCPCB Part # C25804 -> C; Specification 10k 0603 1% 100mW -> 10k 0402 1% 100mW
- R39: footprint cocotter_resistor:r0603_reflow -> cocotter_resistor:r0402_reflow; symbol cocotter_resistors:R_0R_0603 -> cocotter_resistors:R_0R_0402; JLCPCB Part # C431718 -> C; Specification 0R 0603 20mOhms max 100mW -> 0R 0603

Commit message: pmi2023 : corrections after review, digital servo added, battery connector added
Parts:
- R101, R45: footprint cocotter_resistor:r0603_reflow -> cocotter_resistor:r0402_reflow; symbol cocotter_resistors:R_91k_0603_1% -> cocotter_resistors:R_91k_0402_1%; JLCPCB Part # C23265 -> C327323; Specification 91k 0603 1% 100mW -> 91k 0402 1% 100mW; now not fitted
- R125, R126, R127, R129, R130, R131, R38, R44: footprint cocotter_resistor:r0603_reflow -> cocotter_resistor:r0402_reflow; symbol cocotter_resistors:R_91k_0603_1% -> cocotter_resistors:R_91k_0402_1%; JLCPCB Part # C23265 -> C327323; Specification 91k 0603 1% 100mW -> 91k 0402 1% 100mW
- R141: footprint cocotter_resistor:r0603_reflow -> cocotter_resistor:r0402_reflow; symbol cocotter_resistors:R_0R_0603 -> cocotter_resistors:R_0R_0402; JLCPCB Part # C431718 -> C; Specification 0R 0603 20mOhms max 100mW -> 0R 0603
