File: elec/hw/cartes/pmi_2023/interface.kicad_sch (KiCad schematic)
At the start: 41 parts, among them SW3 MSS12C02LS-BB2.0, SW4 TM-4175-B-A, SW5 DS1040-04RN, U11 TCA6408ARGTR, U18 RPI-222N1, U24 SN74LVC2G17DBV, U25 SN74LVC2G17DBV

Commit message: bom updated and component selection optimized to decrease bom cost
Parts:
- R115, R116, R119, R68, R69, R70, R71, R72, R73, R77, R78, R79: value 100k -> 91k 1%; symbol cocotter_resistors:R_100k_0603_1% -> cocotter_resistors:R_91k_0603_1%; JLCPCB Part # C25803 -> C23265; Specification 100k 0603 1% 100mW -> 91k 0603 1% 100mW; mouser 603-RC0603FR-10100KL -> (none)
- SW5: value DS1040-04RN -> HAD-04HWAG-2; footprint cocotter_connectors:DS1040-04RN -> cocotter_connectors:HAD-04HWAG-2; symbol cocotter_connectors:DS1040-04RN -> cocotter_connectors:HAD-04HWAG-2; JLCPCB Part # C3024970 -> C437204
- U18: value RPI-222N1 -> RPI-0352E; footprint cocotter_ic:RPI-222 -> cocotter_ic:RPI-0352E; symbol cocotter_ic:RPI-222N1 -> cocotter_ic:RPI-0352E; JLCPCB Part # C403662 -> C509307
Other:
- moved on the sheet: R115, R118, R68, R69, R71, R72, R77, R78, R79, U18

Commit message: first pass review corrections
Changed lines of the file:
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@@
 		)
 	)
-	(text_box "I2C@ : 0x42"
+	(text_box "I2C@ : 0b0111100 or 0b0111101"
+		(exclude_from_sim no)
+		(at 100.33 184.15 0)
+		(size 13.97 10.16)
+		(stroke
+			(width 0)
+			(type default)
+		)
+		(fill
+			(type color)
+			(color 0 194 0 1)
+		)
+		(effects
+			(font
+				(size 1.27 1.27)
+			)
+		)
+	)
+	(text_box "I2C@ : 0b0100001"
 		(exclude_from_sim no)
 		(at 107.95 64.77 0)
@@
 		(on_board yes)
 		(dnp no)
-		(fields_autoplaced yes)
 		(property "Reference" "SW5"
 			(at 45.72 163.8299 0)
@@
 		)
 		(property "Footprint" "cocotter_connectors:HAD-04HWAG-2"
-			(at 45.72 168.9099 0)
+			(at 33.528 169.672 0)
 			(effects
 				(font
@@
 				)
 				(justify left)
-			)
-		)
+				(hide yes)
+			)
+		)

Commit message: second round of review corrections
Connections:
- net GND_m: now also SW3.MP
Other:
- moved on the sheet: R119
Changed lines of the file:
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@@
 	)
 	(junction
+		(at 111.76 139.7)
+		(diameter 0)
+		(color 0 0 0 0)
+	)
+	(junction
 		(at 194.31 19.05)
 		(diameter 0)
@@
 	)
 	(junction
-		(at 72.39 144.78)
+		(at 134.62 127)
 		(diameter 0)
 		(color 0 0 0 0)
 	)
 	(junction
-		(at 82.55 125.73)
+		(at 72.39 144.78)
 		(diameter 0)
 		(color 0 0 0 0)
 	)
 	(junction
-		(at 220.98 119.38)
+		(at 82.55 125.73)
 		(diameter 0)
 		(color 0 0 0 0)
 	)
 	(junction
-		(at 128.27 127)
+		(at 220.98 119.38)
 		(diameter 0)
 		(color 0 0 0 0)
@@
 	(wire
 		(pts
-			(xy 111.76 124.46) (xy 101.6 124.46)
+			(xy 116.84 124.46) (xy 101.6 124.46)
 		)
 		(stroke
@@
 	(wire
 		(pts
+			(xy 121.92 139.7) (xy 111.76 139.7)
+		)
+		(stroke
+			(width 0)
+			(type default)
+		)
+	)
+	(wire
+		(pts
 			(xy 62.23 128.27) (xy 72.39 128.27)
 		)
@@
 	(wire
 		(pts
-			(xy 53.34 38.1) (xy 53.34 59.69)
+			(xy 121.92 133.35) (xy 121.92 139.7)
 		)
 		(stroke
@@
 	(wire
 		(pts
-			(xy 111.76 132.08) (xy 111.76 129.54)
+			(xy 53.34 38.1) (xy 53.34 59.69)
 		)
 		(stroke
@@
 	(wire
 		(pts
-			(xy 128.27 115.57) (xy 128.27 116.84)
+			(xy 134.62 115.57) (xy 134.62 116.84)
 		)
 		(stroke
@@
 	(wire
 		(pts
-			(xy 121.92 127) (xy 128.27 127)
+			(xy 127 127) (xy 134.62 127)
 		)
 		(stroke
@@
 	(wire
 		(pts
+			(xy 134.62 127) (xy 142.24 127)
+		)
+		(stroke
+			(width 0)
+			(type default)
+		)
+	)
+	(wire
+		(pts
 			(xy 217.17 77.47) (xy 218.44 77.47)
 		)
@@
 	(wire
 		(pts
+			(xy 111.76 129.54) (xy 111.76 132.08)
+		)
+		(stroke
+			(width 0)
+			(type default)
+		)
+	)
+	(wire
+		(pts
 			(xy 62.23 144.78) (xy 69.85 144.78)
 		)
@@
 	(wire
 		(pts
-			(xy 128.27 127) (xy 142.24 127)
-		)
-		(stroke
-			(width 0)
-			(type default)
-		)
-	)
-	(wire
-		(pts
 			(xy 217.17 41.91) (xy 218.44 41.91)
 		)
@@
 	(wire
 		(pts
+			(xy 116.84 129.54) (xy 111.76 129.54)
+		)
+		(stroke
+			(width 0)
+			(type default)
+		)
+	)
+	(wire
+		(pts
 			(xy 20.32 190.5) (xy 30.48 190.5)
 		)
@@
 	(wire
 		(pts
-			(xy 128.27 127) (xy 128.27 124.46)
+			(xy 134.62 127) (xy 134.62 124.46)
 		)
 		(stroke
@@
 	(symbol
 		(lib_id "cocotter_connectors:MSS12C02LS-BB2.0")
-		(at 116.84 127 0)
+		(at 121.92 127 0)
 		(unit 1)
 		(exclude_from_sim no)
@@
 		(fields_autoplaced yes)
 		(property "Reference" "SW3"
-			(at 116.84 118.11 0)
+			(at 121.92 118.11 0)
 			(effects
 				(font
@@
 		)
 		(property "Value" "MSS12C02LS-BB2.0"
-			(at 116.84 120.65 0)
+			(at 121.92 120.65 0)
 			(effects
 				(font
@@
 		)
 		(property "Footprint" "cocotter_connectors:MSS12C02LS-BB2.0"
-			(at 116.84 127 0)
+			(at 121.92 127 0)
 			(effects
 				(font
@@
 		)
 		(property "Datasheet" "https://www.mouser.fr/datasheet/2/910/606_MSS614-1571571.pdf"
-			(at 116.84 132.08 0)
+			(at 121.92 132.08 0)
 			(effects
 				(font
@@
 		)
 		(property "Description" "100mA max, 12Vdc, 10000 cycles"
-			(at 116.84 127 0)
+			(at 121.92 127 0)
 			(effects
 				(font
@@
 		)
 		(property "JLCPCB Part #" "C3008585"
-			(at 115.57 132.08 0)
+			(at 120.65 132.08 0)
 			(effects
 				(font
@@
 		(pin "B"
 		)
+		(pin "MP"
+		)
 		(instances
 			(project "pmi_2023"
@@
 	(symbol
 		(lib_id "pmi_2023_specific:+3V3_m")
-		(at 128.27 115.57 0)
+		(at 134.62 115.57 0)
 		(unit 1)
 		(exclude_from_sim no)
@@
 		(fields_autoplaced yes)
 		(property "Reference" "#PWR058"
-			(at 128.27 119.38 0)
+			(at 134.62 119.38 0)
 			(effects
 				(font
@@
 		)
 		(property "Value" "+3V3_m"
-			(at 128.27 110.49 0)
+			(at 134.62 110.49 0)
 			(effects
 				(font
@@
 		)
 		(property "Footprint" ""
-			(at 128.27 115.57 0)
+			(at 134.62 115.57 0)
 			(effects
 				(font
@@
 		)
 		(property "Datasheet" ""
-			(at 128.27 115.57 0)
+			(at 134.62 115.57 0)
 			(effects
 				(font
@@
 		)
 		(property "Description" "Power symbol creates a global label with name \"+3V3_m\""
-			(at 128.27 115.57 0)
+			(at 134.62 115.57 0)
 			(effects
 				(font
@@
 	(symbol
 		(lib_id "cocotter_resistors:R_91k_0603_1%")
-		(at 128.27 120.65 0)
+		(at 134.62 120.65 0)
 		(unit 1)
 		(exclude_from_sim no)
@@
 		(dnp no)
 		(property "Reference" "R119"
-			(at 129.54 119.38 0)
+			(at 135.89 119.38 0)
 			(effects
 				(font
@@
 		)
 		(property "Value" "91k 1%"
-			(at 133.096 121.92 0)
+			(at 139.446 121.92 0)
 			(effects
 				(font
@@
 		)
 		(property "Footprint" "cocotter_resistor:r0603_reflow"
-			(at 126.492 120.65 90)
+			(at 132.842 120.65 90)
 			(effects
 				(font
@@
 		)
 		(property "Datasheet" "~"
-			(at 128.27 120.65 0)
+			(at 134.62 120.65 0)
 			(effects
 				(font
@@
 		)
 		(property "Description" "Resistor"
-			(at 128.27 120.65 0)
+			(at 134.62 120.65 0)
 			(effects
 				(font
@@
 		)
 		(property "Specification" "91k 0603 1% 100mW"
-			(at 128.27 120.65 0)
+			(at 134.62 120.65 0)
 			(effects
 				(font
@@
 		)
 		(property "mouser" ""
-			(at 128.27 120.65 0)
+			(at 134.62 120.65 0)
 			(effects
 				(font
@@
 		)
 		(property "JLCPCB Part #" "C23265"
-			(at 128.27 120.65 0)
+			(at 134.62 120.65 0)
 			(effects
 				(font
