File: elec/hw/cartes/pmi_2023/boards_interface.kicad_sch (KiCad schematic)
At the start: 4 parts

Commit message: pmi2023 updated
Connections:
- net com/vbatt_mon_3.45V renamed dig_servo_cmd_top_3v3
- net vbatt_mon_3.45V renamed dig_servo_cmd_3v3
Other:
- sheet com ports: added dig_servo_cmd_3v3; removed vbatt_mon_3.45V
- sheet interface ports: added dig_servo_cmd_3v3, scl_tof_3v3, sda_tof_3v3; removed none
Changed lines of the file:
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@@
-	)
-	(junction
-		(at 190.5 97.79)
-		(diameter 0)
-		(color 0 0 0 0)
 	)
 	(junction
@@
 		(color 0 0 0 0)
 	)
+	(junction
+		(at 193.04 97.79)
+		(diameter 0)
+		(color 0 0 0 0)
+	)
 	(wire
 		(pts
@@
 	(wire
 		(pts
-			(xy 190.5 97.79) (xy 198.12 97.79)
-		)
-		(stroke
-			(width 0)
-			(type default)
-		)
-	)
-	(wire
-		(pts
 			(xy 72.39 80.01) (xy 93.98 80.01)
 		)
@@
 	(wire
 		(pts
-			(xy 173.99 57.15) (xy 173.99 90.17)
+			(xy 165.1 58.42) (xy 165.1 90.17)
 		)
 		(stroke
@@
 	(wire
 		(pts
+			(xy 86.36 158.75) (xy 107.95 158.75)
+		)
+		(stroke
+			(width 0)
+			(type default)
+		)
+	)
+	(wire
+		(pts
 			(xy 86.36 113.03) (xy 111.76 113.03)
 		)
@@
 	(wire
 		(pts
-			(xy 198.12 82.55) (xy 190.5 82.55)
+			(xy 86.36 156.21) (xy 107.95 156.21)
+		)
+		(stroke
+			(width 0)
+			(type default)
+		)
+	)
+	(wire
+		(pts
+			(xy 198.12 82.55) (xy 193.04 82.55)
 		)
 		(stroke
@@
 	(wire
 		(pts
-			(xy 156.21 107.95) (xy 198.12 107.95)
-		)
-		(stroke
-			(width 0)
-			(type default)
-		)
-	)
-	(wire
-		(pts
 			(xy 72.39 67.31) (xy 111.76 67.31)
 		)
@@
 	(wire
 		(pts
-			(xy 198.12 90.17) (xy 173.99 90.17)
+			(xy 198.12 90.17) (xy 165.1 90.17)
 		)
 		(stroke
@@
 	(wire
 		(pts
-			(xy 248.92 107.95) (xy 261.62 107.95)
-		)
-		(stroke
-			(width 0)
-			(type default)
-		)
-	)
-	(wire
-		(pts
 			(xy 72.39 64.77) (xy 111.76 64.77)
 		)
@@
 	(wire
 		(pts
+			(xy 248.92 107.95) (xy 271.78 107.95)
+		)
+		(stroke
+			(width 0)
+			(type default)
+		)
+	)
+	(wire
+		(pts
 			(xy 176.53 72.39) (xy 198.12 72.39)
 		)
@@
 	(wire
 		(pts
-			(xy 190.5 82.55) (xy 190.5 97.79)
+			(xy 193.04 82.55) (xy 193.04 97.79)
 		)
 		(stroke
@@
 	(wire
 		(pts
+			(xy 167.64 107.95) (xy 198.12 107.95)
+		)
+		(stroke
+			(width 0)
+			(type default)
+		)
+	)
+	(wire
+		(pts
 			(xy 17.78 137.16) (xy 41.91 137.16)
 		)
@@
 	(wire
 		(pts
-			(xy 190.5 97.79) (xy 190.5 121.92)
+			(xy 193.04 97.79) (xy 193.04 121.92)
 		)
 		(stroke
@@
 	(wire
 		(pts
+			(xy 193.04 97.79) (xy 198.12 97.79)
+		)
+		(stroke
+			(width 0)
+			(type default)
+		)
+	)
+	(wire
+		(pts
 			(xy 156.21 102.87) (xy 198.12 102.87)
 		)
@@
 	(wire
 		(pts
+			(xy 86.36 149.86) (xy 111.76 149.86)
+		)
+		(stroke
+			(width 0)
+			(type default)
+		)
+	)
+	(wire
+		(pts
 			(xy 160.02 114.3) (xy 160.02 62.23)
 		)
@@
 			(width 0)
 			(type default)
+		)
+	)
+	(label "scl_top_tof_3v3"
+		(at 90.17 156.21 0)
+		(effects
+			(font
+				(size 1.27 1.27)
+			)
+			(justify left bottom)
+		)
+	)
+	(label "dig_servo_cmd_top_3v3"
+		(at 167.64 107.95 0)
+		(effects
+			(font
+				(size 1.27 1.27)
+			)
+			(justify left bottom)
 		)
 	)
@@
 		)
 	)
+	(label "dig_servo_cmd_top_3v3"
+		(at 90.17 149.86 0)
+		(effects
+			(font
+				(size 1.27 1.27)
+			)
+			(justify left bottom)
+		)
+	)
 	(label "right_encod_raw_A_3v3"
 		(at 17.78 142.24 0)
@@
 		)
 	)
+	(label "sda_top_tof_3v3"
+		(at 90.17 158.75 0)
+		(effects
+			(font
+				(size 1.27 1.27)
+			)
+			(justify left bottom)
+		)
+	)
 	(label "right_encod_raw_B_3v3"
 		(at 17.78 144.78 0)
+		(effects
+			(font
+				(size 1.27 1.27)
+			)
+			(justify left bottom)
+		)
+	)
+	(label "dig_servo_cmd_3v3"
+		(at 255.27 107.95 0)
 		(effects
 			(font
@@
 		(shape input)
 		(at 261.62 69.85 0)
-		(effects
-			(font
-				(size 1.27 1.27)
-			)
-			(justify left)
-		)
-	)
-	(hierarchical_label "vbatt_mon_3.45V"
-		(shape input)
-		(at 261.62 107.95 0)
 		(effects
 			(font
@@
 	(symbol
 		(lib_id "pmi_2023_specific:GND_m")
-		(at 190.5 121.92 0)
+		(at 193.04 121.92 0)
 		(unit 1)
 		(exclude_from_sim no)
@@
 		(fields_autoplaced yes)
 		(property "Reference" "#PWR091"
-			(at 190.5 128.27 0)
+			(at 193.04 128.27 0)
 			(effects
 				(font
@@
 		)
 		(property "Value" "GND_m"
-			(at 190.5 127 0)
+			(at 193.04 127 0)
 			(effects
 				(font
@@
 		)
 		(property "Footprint" ""
-			(at 190.5 121.92 0)
+			(at 193.04 121.92 0)
 			(effects
 				(font
@@
 		)
 		(property "Datasheet" ""
-			(at 190.5 121.92 0)
+			(at 193.04 121.92 0)
 			(effects
 				(font
@@
 		)
 		(property "Description" "Power symbol creates a global label with name \"GND\" , ground"
-			(at 190.5 121.92 0)
+			(at 193.04 121.92 0)
 			(effects
 				(font
@@
 	(symbol
 		(lib_id "pmi_2023_specific:+3V3_m")
-		(at 173.99 57.15 0)
+		(at 165.1 58.42 0)
 		(unit 1)
 		(exclude_from_sim no)
@@
 		(fields_autoplaced yes)
 		(property "Reference" "#PWR097"
-			(at 173.99 60.96 0)
+			(at 165.1 62.23 0)
 			(effects
 				(font
@@
 		)
 		(property "Value" "+3V3_m"
-			(at 173.99 52.07 0)
+			(at 165.1 53.34 0)
 			(effects
 				(font
@@
 		)
 		(property "Footprint" ""
-			(at 173.99 57.15 0)
+			(at 165.1 58.42 0)
 			(effects
 				(font
@@
 		)
 		(property "Datasheet" ""
-			(at 173.99 57.15 0)
+			(at 165.1 58.42 0)
 			(effects
 				(font
@@
 		)
 		(property "Description" "Power symbol creates a global label with name \"+3V3_m\""
-			(at 173.99 57.15 0)
+			(at 165.1 58.42 0)
 			(effects
 				(font
@@
 	(sheet
 		(at 111.76 38.1)
-		(size 44.45 109.22)
+		(size 44.45 115.57)
 		(exclude_from_sim no)
 		(in_bom yes)
@@
 		)
 		(property "Sheetfile" "com.kicad_sch"
-			(at 111.76 147.9046 0)
+			(at 111.76 154.2546 0)
 			(effects
 				(font
@@
 			)
 		)
-		(pin "vbatt_mon_3.45V" input
-			(at 156.21 107.95 0)
-			(effects
-				(font
-					(size 1.27 1.27)
-				)
-				(justify right)
-			)
-		)
 		(pin "pwm_left" output
 			(at 156.21 102.87 0)
@@
 				)
 				(justify right)
+			)
+		)
+		(pin "dig_servo_cmd_3v3" output
+			(at 111.76 149.86 180)
+			(effects
+				(font
+					(size 1.27 1.27)
+				)
+				(justify left)
 			)
 		)
@@
 	(sheet
 		(at 41.91 106.68)
-		(size 44.45 40.64)
+		(size 44.45 54.61)
 		(exclude_from_sim no)
 		(in_bom yes)
@@
 		)
 		(property "Sheetfile" "interface.kicad_sch"
-			(at 41.91 147.9046 0)
+			(at 41.91 161.8746 0)
 			(effects
 				(font
@@
 			)
 		)
+		(pin "dig_servo_cmd_3v3" input
+			(at 86.36 149.86 0)
+			(effects
+				(font
+					(size 1.27 1.27)
+				)
+				(justify right)
+			)
+		)
+		(pin "scl_tof_3v3" input
+			(at 86.36 156.21 0)
+			(effects
+				(font
+					(size 1.27 1.27)
+				)
+				(justify right)
+			)
+		)
+		(pin "sda_tof_3v3" bidirectional
+			(at 86.36 158.75 0)
+			(effects
+				(font
+					(size 1.27 1.27)
+				)
+				(justify right)
+			)
+		)
