File: elec/hw/cartes/pmi_2023/boards_interface.kicad_sch (KiCad schematic)
At the start: 4 parts

Commit message: pmi2023 : routing updated
Changed lines of the file:
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@@
+		)
+	)
+	(hierarchical_label "vbatt_mon_3.45V"
+		(shape output)
+		(at 278.13 107.95 0)
+		(effects
+			(font
+				(size 1.27 1.27)
+			)
+			(justify left)
 		)
 	)

Commit message: pmi2023 : corrections after review, digital servo added, battery connector added
Parts:
- added R103: 0R, cocotter_resistor:r0402_reflow, symbol cocotter_resistors:R_0R_0402
Connections:
- net dig_servo_cmd_top_3v3: now also R103.1; no longer J49.2 (vbat_mon_4.35V)
- net dig_servo_cmd_3v3 renamed spare
- new net: J49.2 (vbat_mon_4.35V), R103.2
Changed lines of the file:
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@@
 	(wire
 		(pts
-			(xy 86.36 158.75) (xy 107.95 158.75)
+			(xy 86.36 158.75) (xy 102.87 158.75)
+		)
+		(stroke
+			(width 0)
+			(type default)
+		)
+	)
+	(wire
+		(pts
+			(xy 191.77 107.95) (xy 198.12 107.95)
 		)
 		(stroke
@@
 	(wire
 		(pts
-			(xy 86.36 156.21) (xy 107.95 156.21)
+			(xy 86.36 156.21) (xy 102.87 156.21)
 		)
 		(stroke
@@
 	(wire
 		(pts
-			(xy 248.92 107.95) (xy 271.78 107.95)
+			(xy 248.92 107.95) (xy 261.62 107.95)
 		)
 		(stroke
@@
 	(wire
 		(pts
-			(xy 167.64 107.95) (xy 198.12 107.95)
+			(xy 161.29 107.95) (xy 184.15 107.95)
 		)
 		(stroke
@@
 	)
 	(label "scl_top_tof_3v3"
-		(at 90.17 156.21 0)
+		(at 87.63 156.21 0)
 		(effects
 			(font
@@
 	)
 	(label "dig_servo_cmd_top_3v3"
-		(at 167.64 107.95 0)
+		(at 161.29 107.95 0)
 		(effects
 			(font
@@
 	)
 	(label "dig_servo_cmd_top_3v3"
-		(at 90.17 149.86 0)
+		(at 87.63 149.86 0)
 		(effects
 			(font
@@
 	)
 	(label "sda_top_tof_3v3"
-		(at 90.17 158.75 0)
+		(at 87.63 158.75 0)
 		(effects
 			(font
@@
 	(label "right_encod_raw_B_3v3"
 		(at 17.78 144.78 0)
-		(effects
-			(font
-				(size 1.27 1.27)
-			)
-			(justify left bottom)
-		)
-	)
-	(label "dig_servo_cmd_3v3"
-		(at 255.27 107.95 0)
 		(effects
 			(font
@@
 		)
 	)
-	(hierarchical_label "vbatt_mon_3.45V"
+	(hierarchical_label "spare"
 		(shape output)
-		(at 278.13 107.95 0)
+		(at 261.62 107.95 0)
 		(effects
 			(font
@@
 					(unit 1)
 				)
+			)
+		)
+	)
+	(symbol
+		(lib_id "cocotter_resistors:R_0R_0402")
+		(at 187.96 107.95 90)
+		(unit 1)
+		(exclude_from_sim no)
+		(in_bom yes)
+		(on_board yes)
+		(dnp no)
+		(property "Reference" "R103"
+			(at 181.864 109.22 90)
+			(effects
+				(font
+					(size 1.27 1.27)
+				)
+			)
+		)
+		(property "Value" "0R"
+			(at 187.706 107.95 90)
+			(effects
+				(font
+					(size 1.27 1.27)
+				)
+			)
+		)
+		(property "Footprint" "cocotter_resistor:r0402_reflow"
+			(at 187.96 109.728 90)
+			(effects
+				(font
+					(size 1.27 1.27)
+				)
+				(hide yes)
+			)
+		)
+		(property "Datasheet" "~"
+			(at 187.96 107.95 0)
+			(effects
+				(font
+					(size 1.27 1.27)
+				)
+				(hide yes)
+			)
+		)
+		(property "Description" "Resistor"
+			(at 187.96 107.95 0)
+			(effects
+				(font
+					(size 1.27 1.27)
+				)
+				(hide yes)
+			)
+		)
+		(property "Specification" "0R 0603"
+			(at 187.96 107.95 0)
+			(effects
+				(font
+					(size 1.27 1.27)
+				)
+				(hide yes)
+			)
+		)
+		(property "mouser" ""
+			(at 187.96 107.95 0)
+			(effects
+				(font
+					(size 1.27 1.27)
+				)
+				(hide yes)
+			)
+		)
+		(property "JLCPCB Part #" "C"
+			(at 187.96 107.95 0)
+			(effects
+				(font
+					(size 1.27 1.27)
+				)
+				(hide yes)
+			)
+		)
+		(pin "1"
+		)
+		(pin "2"
+		)
+		(instances
+			(project ""
+				(path "/334a657f-c66c-4260-9567-14f1c99913d7/9da1923e-9bb0-4408-8ee2-582c85dcd497"
+					(reference "R103")
+					(unit 1)
+				)
