File: elec/hw/cartes/pmi_2023/pmi_tof_sensor/pmi_tof_sensor.kicad_pcb (KiCad board)
At the start: 2 copper layers, 21 x 23.7 mm, 31 parts, among them J1 tof_sensor_female, Q1 BSS84, Q4 BSS8402DW-7-F, U3 VL53L1CXV0FY1, U4 VL53L5CXV0GC

Commit message: 18nF capacitors replaced by 2nF
Parts:
- C9: value 1nF 50V -> 2nF 50V
- R11, R12, R15, R17, R18: value 100k -> 91k 1%
Changed lines of the file:
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@@
 			)
 		)
-		(property "Value" "100k"
+		(property "Value" "91k 1%"
 			(at 0 -1 0)
 			(unlocked yes)
@@
 			)
 		)
-		(property "Specification" "100k 0603 1% 100mW"
+		(property "Specification" "91k 0603 1% 100mW"
 			(at 0 0 0)
 			(unlocked yes)
@@
 			)
 		)
-		(property "mouser" "603-RC0603FR-10100KL"
+		(property "mouser" ""
 			(at 0 0 0)
 			(unlocked yes)
@@
 			)
 		)
-		(property "JLCPCB" "C25803"
-			(at 0 0 0)
+		(property "JLCPCB Part #" "C23265"
+			(at 0 0 180)
 			(unlocked yes)
 			(layer "B.Fab")
@@
 			)
 		)
-		(property "Value" "100k"
+		(property "Value" "91k 1%"
 			(at 0 -1 180)
 			(unlocked yes)
@@
 			)
 		)
-		(property "Specification" "100k 0603 1% 100mW"
+		(property "Specification" "91k 0603 1% 100mW"
 			(at 0 0 0)
 			(layer "B.Fab")
@@
 			)
 		)
-		(property "mouser" "603-RC0603FR-10100KL"
+		(property "mouser" ""
 			(at 0 0 0)
 			(layer "B.Fab")
@@
 			)
 		)
-		(property "JLCPCB" "C25803"
-			(at 0 0 180)
+		(property "JLCPCB Part #" "C23265"
+			(at 0 0 0)
 			(unlocked yes)
 			(layer "B.Fab")
@@
 			)
 		)
-		(property "Value" "1nF 50V"
+		(property "Value" "2nF 50V"
 			(at 0 -1.43 90)
 			(layer "B.Fab")
@@
 			)
 		)
-		(property "Specification" "1nF 50V X7R 0603 "
+		(property "Specification" "2nF 50V X7R 0603 "
 			(at 0 0 -90)
 			(unlocked yes)
@@
 		(property "JLCPCB" "C1588"
 			(at 0 0 -90)
+			(unlocked yes)
+			(layer "B.Fab")
+			(hide yes)
+			(effects
+				(font
+					(size 1 1)
+					(thickness 0.15)
+				)
+				(justify mirror)
+			)
+		)
+		(property "JLCPCB Part #" "C282245"
+			(at 0 0 90)
 			(unlocked yes)
 			(layer "B.Fab")
@@
 			)
 		)
-		(property "Value" "100k"
+		(property "Value" "91k 1%"
 			(at 0 -1 -90)
 			(unlocked yes)
@@
 			)
 		)
-		(property "Specification" "100k 0603 1% 100mW"
+		(property "Specification" "91k 0603 1% 100mW"
 			(at 0 0 -90)
 			(unlocked yes)
@@
 			)
 		)
-		(property "mouser" "603-RC0603FR-10100KL"
+		(property "mouser" ""
 			(at 0 0 -90)
 			(unlocked yes)
@@
 			)
 		)
-		(property "JLCPCB" "C25803"
-			(at 0 0 -90)
+		(property "JLCPCB Part #" "C23265"
+			(at 0 0 90)
 			(unlocked yes)
 			(layer "B.Fab")
@@
 			)
 		)
-		(property "Value" "100k"
+		(property "Value" "91k 1%"
 			(at 0 -1 90)
 			(unlocked yes)
@@
 			)
 		)
-		(property "Specification" "100k 0603 1% 100mW"
-			(at 0 0 90)
-			(unlocked yes)
-			(layer "B.Fab")
-			(hide yes)
-			(effects
-				(font
-					(size 1 1)
-					(thickness 0.15)
-				)
-				(justify mirror)
-			)
-		)
-		(property "mouser" "603-RC0603FR-10100KL"
-			(at 0 0 90)
-			(unlocked yes)
-			(layer "B.Fab")
-			(hide yes)
-			(effects
-				(font
-					(size 1 1)
-					(thickness 0.15)
-				)
-				(justify mirror)
-			)
-		)
-		(property "JLCPCB" "C25803"
-			(at 0 0 90)
+		(property "Specification" "91k 0603 1% 100mW"
+			(at 0 0 90)
+			(unlocked yes)
+			(layer "B.Fab")
+			(hide yes)
+			(effects
+				(font
+					(size 1 1)
+					(thickness 0.15)
+				)
+				(justify mirror)
+			)
+		)
+		(property "mouser" ""
+			(at 0 0 90)
+			(unlocked yes)
+			(layer "B.Fab")
+			(hide yes)
+			(effects
+				(font
+					(size 1 1)
+					(thickness 0.15)
+				)
+				(justify mirror)
+			)
+		)
+		(property "JLCPCB Part #" "C23265"
+			(at 0 0 -90)
 			(unlocked yes)
 			(layer "B.Fab")
@@
 			)
 		)
-		(property "Value" "100k"
+		(property "Value" "91k 1%"
 			(at 0 -1 180)
 			(unlocked yes)
@@
 			)
 		)
-		(property "Specification" "100k 0603 1% 100mW"
+		(property "Specification" "91k 0603 1% 100mW"
 			(at 0 0 0)
 			(layer "B.Fab")
@@
 			)
 		)
-		(property "mouser" "603-RC0603FR-10100KL"
+		(property "mouser" ""
 			(at 0 0 0)
 			(layer "B.Fab")
@@
 			)
 		)
-		(property "JLCPCB" "C25803"
-			(at 0 0 180)
-			(unlocked yes)
-			(layer "B.Fab")
+		(property "JLCPCB Part #" "C23265"
+			(at 0 0 0)
+			(unlocked yes)
+			(layer "B.Fab")
