File: elec/hw/cartes/sabotter_2026/uc.kicad_sch (KiCad schematic)
At the start: 38 parts, among them J3 USB4120-03-C, SW1 PTS525 SK15 SMTR2 LFS, SW3 DSIC01LSGER, U3 ESP32-S3-WROOM-1

Commit message: sabotter updated after review
Parts:
- added R30, R33, R73, R74, R75, R76: 0R, cocotter_resistor:r0603_reflow, symbol cocotter_resistors:R_0R_0603
- R16, R17: value 390R 1% -> 0R; symbol cocotter_resistors:R_390R_0603_1% -> cocotter_resistors:R_0R_0603; JLCPCB Part # C23151 -> C431718; Specification 390R 0603 1% 100mW -> 0R 0603 20mOhms max 100mW
Connections:
- net encod_mot0_A_3v3: now also R30.1; no longer U3.19 (IO11,RTC_GPIO11,GPIO11,TOUCH11,FSPID,FSPIIO5,SUBSPID)
- net encod_mot0_B_3v3: now also R33.1; no longer U3.20 (IO12,RTC_GPIO12,GPIO12,TOUCH12,FSPICLK,FSPIIO6,SUBSPICLK)
- net encod_mot1_A_3v3: now also R76.1; no longer U3.9 (IO16,RTC_GPIO16,GPIO16,U0CTS,XTAL_32K_N)
- net encod_mot1_B_3v3: now also R75.1; no longer U3.8 (IO15,RTC_GPIO15,GPIO15,U0RTS,XTAL_32K_P)
- net encod_mot2_A_3v3: now also R74.1; no longer U3.22 (IO14,RTC_GPIO14,GPIO14,TOUCH14,FSPIWP,FSPIDQS,SUBSPIWP)
- net encod_mot2_B_3v3: now also R73.1; no longer U3.21 (IO13,RTC_GPIO13,GPIO13,TOUCH13,FSPIQ,FSPIIO7,SUBSPIQ)
- new net: R30.2, U3.19 (IO11,RTC_GPIO11,GPIO11,TOUCH11,FSPID,FSPIIO5,SUBSPID)
- new net: R33.2, U3.20 (IO12,RTC_GPIO12,GPIO12,TOUCH12,FSPICLK,FSPIIO6,SUBSPICLK)
- new net: R73.2, U3.21 (IO13,RTC_GPIO13,GPIO13,TOUCH13,FSPIQ,FSPIIO7,SUBSPIQ)
- new net: R74.2, U3.22 (IO14,RTC_GPIO14,GPIO14,TOUCH14,FSPIWP,FSPIDQS,SUBSPIWP)
- new net: R75.2, U3.8 (IO15,RTC_GPIO15,GPIO15,U0RTS,XTAL_32K_P)
- new net: R76.2, U3.9 (IO16,RTC_GPIO16,GPIO16,U0CTS,XTAL_32K_N)

Commit message: jlcpcb part added
Parts:
- J3: JLC C7450621 -> (none); JLCPCB Part # (none) -> C7450621
