File: elec/hw/cartes/sabotter_2026/sensors.kicad_sch (KiCad schematic)
At the start: 30 parts, among them J5 2-1445055-4, U4 ADXRS453BRGZ, U5 SCH16T-K01-10

Commit message: sabotter wip
Parts:
- removed J5: 2-1445055-4, cocotter_connectors:2-1445055-4, symbol cocotter_connectors:2-1445055-4
- added J17: 22272061, cocotter_connectors:22272061, symbol cocotter_connectors:22272061
- added J5: 22272041, cocotter_connectors:22272041, symbol cocotter_connectors:22272041
- added R64: 91k 1%, cocotter_resistor:r0603_reflow, symbol cocotter_resistors:R_91k_0603_1%
- R36: value 91k 1% -> 10k 1%; symbol cocotter_resistors:R_91k_0603_1% -> cocotter_resistors:R_10k_0603_1%; JLCPCB Part # C23265 -> C25804; Specification 91k 0603 1% 100mW -> 10k 0603 1% 100mW; mouser (none) -> 603-RC0603FR-10100KL; now not fitted
Connections:
- net +3V3: now also J17.6, R64.1
- net +5V: now also J5.4
- net GND: now also J17.1, J5.1
- net gyro_miso_3v3: now also J17.4
- net gyro_mosi_3v3: now also J17.3
- net gyro_sck_3v3: now also J17.2
- net lidar_pwm_3v3: now also J5.2
- net lidar_rx_3v3: now also J5.3
- net /gyro_cs_3v3: now also J17.5, R64.2
Other:
- moved on the sheet: C16, C17, C18, C19, C20, R35, R37, R38, TP4, TP5, U5

Commit message: sabotter wip
Connections:
- net GND: now also J5.3; no longer J5.1
- net lidar_rx_3v3: now also J5.1; no longer J5.3, R28.2, R30.2
- new net lidar_tx_3v3: R28.2, R30.2
Other:
- moved on the sheet: J5, R32
Changed lines of the file:
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@@
 	)
 	(junction
+		(at 80.01 118.11)
+		(diameter 0)
+		(color 0 0 0 0)
+	)
+	(junction
 		(at 204.47 73.66)
 		(diameter 0)
@@
 	)
 	(junction
-		(at 73.66 115.57)
-		(diameter 0)
-		(color 0 0 0 0)
-	)
-	(junction
 		(at 168.91 19.05)
 		(diameter 0)
@@
 	)
 	(junction
+		(at 73.66 120.65)
+		(diameter 0)
+		(color 0 0 0 0)
+	)
+	(junction
 		(at 179.07 73.66)
 		(diameter 0)
@@
 	)
 	(junction
-		(at 73.66 118.11)
-		(diameter 0)
-		(color 0 0 0 0)
-	)
-	(junction
 		(at 72.39 74.93)
 		(diameter 0)
@@
 	)
 	(junction
-		(at 73.66 127)
+		(at 196.85 73.66)
 		(diameter 0)
 		(color 0 0 0 0)
 	)
 	(junction
-		(at 196.85 73.66)
+		(at 60.96 99.06)
 		(diameter 0)
 		(color 0 0 0 0)
 	)
 	(junction
-		(at 60.96 99.06)
+		(at 80.01 132.08)
 		(diameter 0)
 		(color 0 0 0 0)
@@
 	(wire
 		(pts
-			(xy 227.33 25.4) (xy 245.11 25.4)
+			(xy 30.48 120.65) (xy 73.66 120.65)
 		)
 		(stroke
@@
 	(wire
 		(pts
-			(xy 204.47 73.66) (xy 207.01 73.66)
+			(xy 227.33 25.4) (xy 245.11 25.4)
 		)
 		(stroke
@@
 	(wire
 		(pts
-			(xy 203.2 24.13) (xy 203.2 17.78)
+			(xy 204.47 73.66) (xy 207.01 73.66)
 		)
 		(stroke
@@
 	(wire
 		(pts
-			(xy 203.2 17.78) (xy 205.74 17.78)
+			(xy 203.2 24.13) (xy 203.2 17.78)
 		)
 		(stroke
@@
 	(wire
 		(pts
-			(xy 168.91 69.85) (xy 168.91 73.66)
+			(xy 203.2 17.78) (xy 205.74 17.78)
 		)
 		(stroke
@@
 	(wire
 		(pts
-			(xy 73.66 109.22) (xy 73.66 115.57)
+			(xy 168.91 69.85) (xy 168.91 73.66)
 		)
 		(stroke
@@
 	(wire
 		(pts
-			(xy 40.64 115.57) (xy 73.66 115.57)
-		)
-		(stroke
-			(width 0)
-			(type default)
-		)
-	)
-	(wire
-		(pts
 			(xy 68.58 177.8) (xy 86.36 177.8)
 		)
@@
 	(wire
 		(pts
+			(xy 80.01 130.81) (xy 80.01 132.08)
+		)
+		(stroke
+			(width 0)
+			(type default)
+		)
+	)
+	(wire
+		(pts
 			(xy 85.09 74.93) (xy 87.63 74.93)
 		)
@@
 	(wire
 		(pts
-			(xy 13.97 85.09) (xy 111.76 85.09)
+			(xy 30.48 118.11) (xy 80.01 118.11)
 		)
 		(stroke
 			(width 0)
-			(type dash)
+			(type default)
 		)
 	)
 	(wire
 		(pts
-			(xy 45.72 127) (xy 45.72 120.65)
+			(xy 13.97 85.09) (xy 111.76 85.09)
 		)
 		(stroke
 			(width 0)
-			(type default)
+			(type dash)
 		)
 	)
@@
 	(wire
 		(pts
-			(xy 40.64 118.11) (xy 73.66 118.11)
-		)
-		(stroke
-			(width 0)
-			(type default)
-		)
-	)
-	(wire
-		(pts
 			(xy 217.17 36.83) (xy 218.44 36.83)
 		)
@@
 	(wire
 		(pts
-			(xy 95.25 115.57) (xy 73.66 115.57)
+			(xy 95.25 120.65) (xy 73.66 120.65)
 		)
 		(stroke
@@
 	(wire
 		(pts
+			(xy 35.56 132.08) (xy 80.01 132.08)
+		)
+		(stroke
+			(width 0)
+			(type default)
+		)
+	)
+	(wire
+		(pts
 			(xy 207.01 71.12) (xy 207.01 73.66)
 		)
@@
 	(wire
 		(pts
-			(xy 73.66 130.81) (xy 73.66 127)
+			(xy 80.01 134.62) (xy 80.01 132.08)
 		)
 		(stroke
@@
 	(wire
 		(pts
-			(xy 218.44 54.61) (xy 224.79 54.61)
+			(xy 30.48 113.03) (xy 45.72 113.03)
 		)
 		(stroke
@@
 	(wire
 		(pts
-			(xy 82.55 74.93) (xy 85.09 74.93)
+			(xy 218.44 54.61) (xy 224.79 54.61)
 		)
 		(stroke
@@
 	(wire
 		(pts
-			(xy 77.47 74.93) (xy 82.55 74.93)
+			(xy 82.55 74.93) (xy 85.09 74.93)
 		)
 		(stroke
@@
 	(wire
 		(pts
-			(xy 45.72 120.65) (xy 40.64 120.65)
+			(xy 77.47 74.93) (xy 82.55 74.93)
 		)
 		(stroke
@@
 	(wire
 		(pts
-			(xy 73.66 118.11) (xy 73.66 119.38)
+			(xy 80.01 118.11) (xy 80.01 123.19)
 		)
 		(stroke
@@
 	(wire
 		(pts
-			(xy 73.66 127) (xy 45.72 127)
+			(xy 30.48 115.57) (xy 35.56 115.57)
 		)
 		(stroke
@@
 	(wire
 		(pts
+			(xy 35.56 115.57) (xy 35.56 132.08)
+		)
+		(stroke
+			(width 0)
+			(type default)
+		)
+	)
+	(wire
+		(pts
 			(xy 156.21 46.99) (xy 184.15 46.99)
 		)
@@
 	(wire
 		(pts
-			(xy 87.63 118.11) (xy 73.66 118.11)
+			(xy 87.63 118.11) (xy 80.01 118.11)
 		)
 		(stroke
@@
 	(wire
 		(pts
-			(xy 45.72 113.03) (xy 40.64 113.03)
+			(xy 73.66 109.22) (xy 73.66 120.65)
 		)
 		(stroke
@@
 	(text "confirmer tension sur LIDAR LD06"
 		(exclude_from_sim no)
-		(at 36.576 135.382 0)
+		(at 34.798 140.462 0)
 		(effects
 			(font
@@
 		)
 	)
-	(label "lidar_tx_3v3"
-		(at 43.18 115.57 0)
+	(label "lidar_rx_3v3"
+		(at 43.18 120.65 0)
 		(effects
 			(font
@@
 	(hierarchical_label "lidar_rx_3v3"
 		(shape output)
-		(at 95.25 115.57 0)
+		(at 95.25 120.65 0)
 		(effects
 			(font
@@
 	(symbol
 		(lib_id "power:GND")
-		(at 73.66 130.81 0)
+		(at 80.01 134.62 0)
 		(mirror y)
 		(unit 1)
@@
 		(dnp no)
 		(property "Reference" "#PWR34"
-			(at 73.66 137.16 0)
+			(at 80.01 140.97 0)
 			(effects
 				(font
@@
 		)
 		(property "Value" "GND"
-			(at 73.66 134.874 0)
+			(at 80.01 138.684 0)
 			(effects
 				(font
@@
 		)
 		(property "Footprint" ""
-			(at 73.66 130.81 0)
+			(at 80.01 134.62 0)
 			(effects
 				(font
@@
 		)
 		(property "Datasheet" ""
-			(at 73.66 130.81 0)
+			(at 80.01 134.62 0)
 			(effects
 				(font
@@
 		)
 		(property "Description" "Power symbol creates a global label with name \"GND\" , ground"
-			(at 73.66 130.81 0)
+			(at 80.01 134.62 0)
 			(effects
 				(font
@@
 	(symbol
 		(lib_id "cocotter_connectors:22272041")
-		(at 40.64 118.11 0)
+		(at 30.48 118.11 0)
 		(unit 1)
 		(exclude_from_sim no)
@@
 		(fields_autoplaced yes)
 		(property "Reference" "J5"
-			(at 36.83 105.41 0)
+			(at 26.67 105.41 0)
 			(effects
 				(font
@@
 		)
 		(property "Value" "22272041"
-			(at 36.83 107.95 0)
+			(at 26.67 107.95 0)
 			(effects
 				(font
@@
 		)
 		(property "Footprint" "cocotter_connectors:22272041"
-			(at 37.338 130.048 0)
+			(at 27.178 130.048 0)
 			(effects
 				(font
@@
 		)
 		(property "Datasheet" "https://www.molex.com/en-us/products/part-detail/22272041"
-			(at 40.64 127 0)
+			(at 30.48 127 0)
 			(effects
 				(font
@@
 		)
 		(property "Description" "mini kk 4 voies vertical"
-			(at 40.64 127 0)
+			(at 30.48 127 0)
 			(effects
 				(font
@@
 	(symbol
 		(lib_id "cocotter_resistors:R_91k_0603_1%")
-		(at 73.66 123.19 0)
+		(at 80.01 127 0)
 		(unit 1)
 		(exclude_from_sim no)
@@
 		(fields_autoplaced yes)
 		(property "Reference" "R32"
-			(at 76.2 121.9199 0)
+			(at 82.55 125.7299 0)
 			(effects
 				(font
@@
 		)
 		(property "Value" "91k 1%"
-			(at 76.2 124.4599 0)
+			(at 82.55 128.2699 0)
 			(effects
 				(font
@@
 		)
 		(property "Footprint" "cocotter_resistor:r0603_reflow"
-			(at 71.882 123.19 90)
+			(at 78.232 127 90)
 			(effects
 				(font
@@
 		)
 		(property "Datasheet" "~"
-			(at 73.66 123.19 0)
+			(at 80.01 127 0)
 			(effects
 				(font
@@
 		)
 		(property "Description" "Resistor"
-			(at 73.66 123.19 0)
+			(at 80.01 127 0)
 			(effects
 				(font
@@
 		)
 		(property "Specification" "91k 0603 1% 100mW"
-			(at 73.66 123.19 0)
+			(at 80.01 127 0)
 			(effects
 				(font
@@
 		)
 		(property "mouser" ""
-			(at 73.66 123.19 0)
+			(at 80.01 127 0)
 			(effects
 				(font
@@
 		)
 		(property "JLCPCB Part #" "C23265"
-			(at 73.66 123.19 0)
+			(at 80.01 127 0)
 			(effects
 				(font

Commit message: sabotter ready for first schematic and routing review
Parts:
- R30, R33: now not fitted
Connections:
- net lidar_tx_3v3 is gone; now on net lidar_pwm_3v3: R28.2, R30.2
- net lidar_pwm_3v3: no longer R29.2, R33.2
- net lidar_rx_3v3: now also R29.2, R33.2
Other:
- note added: "consumption : 300mA at startup 180mA at work"
- moved on the sheet: R28
Changed lines of the file:
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@@
 	(wire
 		(pts
-			(xy 68.58 177.8) (xy 86.36 177.8)
+			(xy 68.58 177.8) (xy 93.98 177.8)
 		)
 		(stroke
@@
 	(wire
 		(pts
-			(xy 63.5 177.8) (xy 68.58 177.8)
+			(xy 62.23 177.8) (xy 68.58 177.8)
 		)
 		(stroke
@@
 	(wire
 		(pts
-			(xy 81.28 180.34) (xy 86.36 180.34)
+			(xy 81.28 180.34) (xy 93.98 180.34)
 		)
 		(stroke
@@
 	(wire
 		(pts
-			(xy 34.29 177.8) (xy 55.88 177.8)
+			(xy 34.29 177.8) (xy 54.61 177.8)
 		)
 		(stroke
@@
 		)
 	)
+	(text "consumption :\n  300mA at startup\n  180mA at work"
+		(exclude_from_sim no)
+		(at 23.876 95.504 0)
+		(effects
+			(font
+				(size 1.27 1.27)
+			)
+		)
+	)
 	(text "LIDAR (LD06)"
 		(exclude_from_sim no)
@@
 		)
 	)
-	(label "lidar_tx_3v3"
-		(at 83.82 177.8 0)
+	(label "lidar_rx_3v3"
+		(at 83.82 180.34 0)
 		(effects
 			(font
@@
 		)
 	)
+	(label "lidar_pwm_3v3"
+		(at 83.82 177.8 0)
+		(effects
+			(font
+				(size 1.27 1.27)
+			)
+			(justify left bottom)
+		)
+	)
 	(label "{slash}gyro_cs_3v3"
 		(at 271.78 58.42 180)
@@
 		)
 	)
-	(label "lidar_pwm_3v3"
-		(at 83.82 180.34 0)
-		(effects
-			(font
-				(size 1.27 1.27)
-			)
-			(justify left bottom)
-		)
-	)
 	(label "gyro_miso_3v3"
 		(at 271.78 60.96 180)
@@
 		(in_bom yes)
 		(on_board yes)
-		(dnp no)
+		(dnp yes)
 		(fields_autoplaced yes)
 		(property "Reference" "R33"
@@
 		(in_bom yes)
 		(on_board yes)
-		(dnp no)
+		(dnp yes)
 		(fields_autoplaced yes)
 		(property "Reference" "R30"
@@
 	(symbol
 		(lib_id "cocotter_resistors:R_0R_0603")
-		(at 59.69 177.8 90)
+		(at 58.42 177.8 90)
 		(unit 1)
 		(exclude_from_sim no)
@@
 		(dnp no)
 		(property "Reference" "R28"
-			(at 59.69 175.514 90)
+			(at 58.42 175.514 90)
 			(effects
 				(font
@@
 		)
 		(property "Value" "0R"
-			(at 59.69 177.8 90)
+			(at 58.42 177.8 90)
 			(effects
 				(font
@@
 		)
 		(property "Footprint" "cocotter_resistor:r0603_reflow"
-			(at 59.69 179.578 90)
+			(at 58.42 179.578 90)
 			(effects
 				(font
@@
 		)
 		(property "Datasheet" "~"
-			(at 59.69 177.8 0)
+			(at 58.42 177.8 0)
 			(effects
 				(font
@@
 		)
 		(property "Description" "Resistor"
-			(at 59.69 177.8 0)
+			(at 58.42 177.8 0)
 			(effects
 				(font
@@
 		)
 		(property "Specification" "0R 0603 20mOhms max 100mW"
-			(at 59.69 177.8 0)
+			(at 58.42 177.8 0)
 			(effects
 				(font
@@
 		)
 		(property "mouser" ""
-			(at 59.69 177.8 0)
+			(at 58.42 177.8 0)
 			(effects
 				(font
@@
 		)
 		(property "JLCPCB Part #" "C431718"
-			(at 59.69 177.8 0)
+			(at 58.42 177.8 0)
 			(effects
 				(font

Commit message: sabotter corrected after review
Parts:
- removed C11, C13, C14, C18, C20: 1µF 50V, cocotter_capacitors:C_0805_2012Metric, symbol cocotter_capacitors:C_1µF_50V_0805
- removed C15, C16, C19: 100nF 50V, cocotter_capacitors:C_0603_1608Metric, symbol cocotter_capacitors:C_100nF_50V_0603
- removed C17: 10µF 25V, cocotter_capacitors:C_0805_2012Metric, symbol cocotter_capacitors:C_10µF_25V_0805_X5R
- removed D5: 1N5819WS, cocotter_diodes:D_SOD-323, symbol cocotter_diodes:1N5819WS
- removed L1: 470µH, cocotter_inductors:L_Kyocera_07A7_7.3x6.6mm, symbol cocotter_inductors:B82422H1474J
- removed R27: 100k, cocotter_resistor:r0603_reflow, symbol cocotter_resistors:R_100k_0603_1%
- removed R35: 91k 1%, cocotter_resistor:r0603_reflow, symbol cocotter_resistors:R_91k_0603_1%
- removed R36: 10k 1%, cocotter_resistor:r0603_reflow, symbol cocotter_resistors:R_10k_0603_1%
- removed R37, R38: 0R, cocotter_resistor:r0603_reflow, symbol cocotter_resistors:R_0R_0603
- removed TP4, TP5: TestPoint, cocotter_others:testpoint-THT-0.5mm, symbol cocotter_others:TestPoint
- removed U4: ADXRS453BRGZ, cocotter_ic:SOIC-16W_7.5x10.3mm_P1.27mm, symbol cocotter_ic:ADXRS453BRGZ
- removed U5: SCH16T-K01-10, cocotter_ic:SCH16T, symbol cocotter_ic:SCH16T-K01-10
- R30, R31, R32, R33, R34, R64: value 91k 1% -> 100k; symbol cocotter_resistors:R_91k_0603_1% -> cocotter_resistors:R_100k_0603_1%; JLCPCB Part # C23265 -> C25803; Specification 91k 0603 1% 100mW -> 100k 0603 1% 100mW; mouser (none) -> 603-RC0603FR-10100KL
Other:
- note removed: "TODO : EXT dry_sync et EXT_RESET"
- moved on the sheet: J17, R64

Commit message: sabotter updated after review
Parts:
- removed R30, R33: 100k, cocotter_resistor:r0603_reflow, symbol cocotter_resistors:R_100k_0603_1%
- added R38, R72: 0R, cocotter_resistor:r0603_reflow, symbol cocotter_resistors:R_0R_0603
Connections:
- net lidar_pwm_3v3: now also R72.2; no longer J5.2
- net lidar_rx_3v3: now also R38.2; no longer J5.1
- new net: J5.2, R72.1
- new net: J5.1, R38.1

Commit message: jlcpcb part added
Parts:
- J17: JLCPCB Part # (none) -> C504992
- J4: value ~ -> 188275-4; JLCPCB Part # (none) -> C720206
- J5: JLCPCB Part # (none) -> C504991
Changed lines of the file:
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@@
 			)
 		)
-		(property "Value" "~"
+		(property "Value" "188275-4"
 			(at 34.29 189.23 0)
 			(effects
@@
 			)
 		)
-		(property "Description" ""
+		(property "Description" "micromatch 4 voies, cms , 188275-4"
 			(at 34.29 189.23 0)
 			(effects
@@
 			)
 		)
+		(property "JLCPCB Part #" "C720206"
+			(at 34.29 180.34 0)
+			(effects
+				(font
+					(size 1.27 1.27)
+				)
+				(hide yes)
+			)
+		)
+		(property "MOUSER" ""
+			(at 34.29 180.34 0)
+			(effects
+				(font
+					(size 1.27 1.27)
+				)
+				(hide yes)
+			)
+		)
 		(pin "1"
 		)
@@
 		)
 		(pin "4"
+		)
+		(pin "3"
 		)
 		(instances
@@
 			)
 		)
+		(property "MOUSER" ""
+			(at 60.96 102.87 0)
+			(effects
+				(font
+					(size 1.27 1.27)
+				)
+				(hide yes)
+			)
+		)
 		(pin "2"
 		)
@@
 			)
 		)
+		(property "MOUSER" ""
+			(at 64.77 180.34 0)
+			(effects
+				(font
+					(size 1.27 1.27)
+				)
+				(hide yes)
+			)
+		)
 		(pin "1"
 		)
@@
 		)
 		(property "JLCPCB Part #" "C25803"
+			(at 73.66 105.41 0)
+			(effects
+				(font
+					(size 1.27 1.27)
+				)
+				(hide yes)
+			)
+		)
+		(property "MOUSER" ""
 			(at 73.66 105.41 0)
 			(effects
@@
 			)
 		)
+		(property "MOUSER" ""
+			(at 87.63 105.41 0)
+			(effects
+				(font
+					(size 1.27 1.27)
+				)
+				(hide yes)
+			)
+		)
 		(pin "2"
 		)
@@
 			)
 		)
+		(property "MOUSER" ""
+			(at 43.18 118.11 0)
+			(effects
+				(font
+					(size 1.27 1.27)
+				)
+				(hide yes)
+			)
+		)
 		(pin "1"
 		)
@@
 		(dnp no)
 		(property "Reference" "J17"
-			(at 172.466 113.03 0)
-			(effects
-				(font
-					(size 1.27 1.27)
-				)
-				(justify right)
+			(at 177.292 113.284 0)
+			(effects
+				(font
+					(size 1.27 1.27)
+				)
 			)
 		)
 		(property "Value" "22272061"
-			(at 170.434 133.35 0)
-			(effects
-				(font
-					(size 1.27 1.27)
-				)
-				(justify right)
+			(at 177.038 133.096 0)
+			(effects
+				(font
+					(size 1.27 1.27)
+				)
 			)
 		)
@@
 		(property "Description" "mini kk 6 voies vertical"
 			(at 171.45 133.35 0)
+			(effects
+				(font
+					(size 1.27 1.27)
+				)
+				(hide yes)
+			)
+		)
+		(property "JLCPCB Part #" "C504992"
+			(at 171.45 124.46 0)
+			(effects
+				(font
+					(size 1.27 1.27)
+				)
+				(hide yes)
+			)
+		)
+		(property "MOUSER" ""
+			(at 171.45 124.46 0)
 			(effects
 				(font
@@
 			)
 		)
+		(property "JLCPCB Part #" "C504991"
+			(at 30.48 118.11 0)
+			(effects
+				(font
+					(size 1.27 1.27)
+				)
+				(hide yes)
+			)
+		)
+		(property "MOUSER" ""
+			(at 30.48 118.11 0)
+			(effects
+				(font
+					(size 1.27 1.27)
+				)
+				(hide yes)
+			)
+		)
 		(pin "1"
 		)
@@
 			)
 		)
+		(property "MOUSER" ""
+			(at 80.01 127 0)
+			(effects
+				(font
+					(size 1.27 1.27)
+				)
+				(hide yes)
+			)
+		)
 		(pin "2"
 		)
@@
 			)
 		)
+		(property "MOUSER" ""
+			(at 58.42 177.8 0)
+			(effects
+				(font
+					(size 1.27 1.27)
+				)
+				(hide yes)
+			)
+		)
 		(pin "1"
 		)
@@
 		)
 		(property "JLCPCB Part #" "C431718"
+			(at 43.18 120.65 0)
+			(effects
+				(font
+					(size 1.27 1.27)
+				)
+				(hide yes)
+			)
+		)
+		(property "MOUSER" ""
 			(at 43.18 120.65 0)
 			(effects
@@
 			(at 153.67 111.76 0)
 			(effects
+				(font
+					(size 1.27 1.27)
+				)
+				(hide yes)
+			)
+		)
+		(property "MOUSER" ""
+			(at 153.67 111.76 0)
+			(effects
