File: elec/hw/cartes/sabotter_2026/supply.kicad_sch (KiCad schematic)
At the start: 21 parts, among them U1 OKI-78SR-3.3/1.5-W36H-C, U2 OKI-78SR-5/1.5-W36H-C

Commit message: sabotter wip
Parts:
- removed H5: MOUNT-PAD-ROUND3.3, cocotter_others:MountingHole_3.2mm_M3_Pad_Via, symbol cocotter_others:MountingHole_Pad_M3
- J1: value ~ -> 22272021
Other:
- moved on the sheet: J1

Commit message: sabotter corrected after review
Parts:
- removed D3: 1N5819WS, cocotter_diodes:D_SOD-323, symbol cocotter_diodes:1N5819WS
- removed R1: 22k 1%, cocotter_resistor:r0603_reflow, symbol cocotter_resistors:R_22k_0603_1%
- added D3: BZT52C3V0S, cocotter_diodes:SOD-323, symbol cocotter_diodes:BZT52C3V0S
- added R1, R27, R35, R36: 100k, cocotter_resistor:r0603_reflow, symbol cocotter_resistors:R_100k_0603_1%
- R2: value 91k 1% -> 100k; symbol cocotter_resistors:R_91k_0603_1% -> cocotter_resistors:R_100k_0603_1%; JLCPCB Part # C23265 -> C25803; Specification 91k 0603 1% 100mW -> 100k 0603 1% 100mW; mouser (none) -> 603-RC0603FR-10100KL
Connections:
- net GND: now also D2.C, D3.2 (A)
- net esp32_vbatt_mon_3v1: now also D3.1 (K)
- net at C1.1, C2.1, C4.1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: now also R1.1, R27.1, R35.1, R36.1; no longer D2.A
- new net: D2.A, R1.2, R27.2, R35.2, R36.2
Other:
- moved on the sheet: D1, D2, J1

Commit message: jlcpcb part added
Parts:
- C6, C7: value 22µF 16V -> 22µF 25V; symbol cocotter_capacitors:C_22µF_16V_1206_X5R -> cocotter_capacitors:C_22µF_25V_1206_X7R; JLCPCB Part # (none) -> C2918511; Specification 10µF 16V X7R 0805 -> 22µF 25V X7R 1206
- J1: JLCPCB Part # (none) -> C293316
