File: elec/hw/cartes/meca_extension_2026/channel.kicad_sch (KiCad schematic)
At the start: 22 parts, among them J2 22272021, J20 5264-3P, J24 22053031, J3 22272021, J4 22053051, Q1 SI2310, Q2 SI2310, Q3 2N7002, U4 TLV9061IDBVR

Commit message: meca_extension : connectors placement modified
Parts:
- removed J2: 22272021, cocotter_connectors:22272021, symbol cocotter_connectors:22272021
- removed J20: 5264-3P, cocotter_connectors:5264-3P, symbol cocotter_connectors:feetech_servo
- added J17: 5267-3P, cocotter_connectors:5267-3P, symbol cocotter_connectors:feetech_servo-V
- added J2: B2B-XH-A, cocotter_connectors:B2B-XH-A, symbol cocotter_connectors:B2B-XH-A
Connections:
- net +6V: now also J17.2 (VCC)
- net +BATT: now also J2.1
- net GND: now also J17.1 (GND)
- net digital_servo_cmd_3v3: now also J17.3 (SIG)
- net at D1.2 (A), Q1.3 (D): now also J2.2
Changed lines of the file:
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@@
+	)
+	(symbol
+		(lib_id "cocotter_connectors:B2B-XH-A")
+		(at 96.52 33.02 180)
+		(unit 1)
+		(exclude_from_sim no)
+		(in_bom yes)
+		(on_board yes)
+		(dnp no)
+		(fields_autoplaced yes)
+		(property "Reference" "J2"
+			(at 104.14 30.4799 0)
+			(effects
+				(font
+					(size 1.27 1.27)
+				)
+				(justify right)
+			)
+		)
+		(property "Value" "B2B-XH-A"
+			(at 104.14 33.0199 0)
+			(effects
+				(font
+					(size 1.27 1.27)
+				)
+				(justify right)
+			)
+		)
+		(property "Footprint" "cocotter_connectors:B2B-XH-A"
+			(at 99.822 21.082 0)
+			(effects
+				(font
+					(size 1.27 1.27)
+				)
+				(hide yes)
+			)
+		)
+		(property "Datasheet" "https://www.jst.fr/core/file.get?path=doc/jst/family/pdf/exh0125.pdf"
+			(at 96.52 24.13 0)
+			(effects
+				(font
+					(size 1.27 1.27)
+				)
+				(hide yes)
+			)
+		)
+		(property "Description" "JST XH 2 voies vertical"
+			(at 96.52 24.13 0)
+			(effects
+				(font
+					(size 1.27 1.27)
+				)
+				(hide yes)
+			)
+		)
+		(property "JLCPCB Part #" "C293316"
+			(at 100.838 23.876 0)
+			(effects
+				(font
+					(size 1.27 1.27)
+				)
+				(hide yes)
+			)
+		)
+		(pin "2"
+		)
+		(pin "1"
+		)
+		(instances
+			(project ""
+				(path "/f6dc6b20-ab52-4b2b-893a-1fb4f3ec4277/067947e6-d018-482f-a78c-eeb83d8dcdcb"
+					(reference "J8")
+					(unit 1)
+				)
+				(path "/f6dc6b20-ab52-4b2b-893a-1fb4f3ec4277/2caf5ca5-b8be-49ab-9f25-cabd53014211"
+					(reference "J5")
+					(unit 1)
+				)
+				(path "/f6dc6b20-ab52-4b2b-893a-1fb4f3ec4277/a1cde7f5-363d-4f36-b502-090ba61d1d03"
+					(reference "J11")
+					(unit 1)
+				)
+				(path "/f6dc6b20-ab52-4b2b-893a-1fb4f3ec4277/cd773c3d-c05b-4eb4-90a6-abf942da4e0b"
+					(reference "J2")
+					(unit 1)
+				)
+			)
+		)
 	)
 	(symbol
@@
 	)
 	(symbol
-		(lib_id "cocotter_connectors:22272021")
-		(at 96.52 33.02 180)
-		(unit 1)
-		(exclude_from_sim no)
-		(in_bom yes)
-		(on_board yes)
-		(dnp no)
-		(fields_autoplaced yes)
-		(property "Reference" "J2"
-			(at 104.14 30.4799 0)
-			(effects
-				(font
-					(size 1.27 1.27)
-				)
-				(justify right)
-			)
-		)
-		(property "Value" "22272021"
-			(at 104.14 33.0199 0)
-			(effects
-				(font
-					(size 1.27 1.27)
-				)
-				(justify right)
-			)
-		)
-		(property "Footprint" "cocotter_connectors:22272021"
-			(at 99.822 21.082 0)
-			(effects
-				(font
-					(size 1.27 1.27)
-				)
-				(hide yes)
-			)
-		)
-		(property "Datasheet" "https://www.molex.com/en-us/products/part-detail/22272021"
-			(at 96.52 24.13 0)
-			(effects
-				(font
-					(size 1.27 1.27)
-				)
-				(hide yes)
-			)
-		)
-		(property "Description" "mini kk 2 voies vertical"
-			(at 96.52 24.13 0)
-			(effects
-				(font
-					(size 1.27 1.27)
-				)
-				(hide yes)
-			)
-		)
-		(property "JLCPCB Part #" "C293316"
-			(at 100.838 23.876 0)
-			(effects
-				(font
-					(size 1.27 1.27)
-				)
-				(hide yes)
-			)
-		)
-		(pin "2"
-		)
-		(pin "1"
-		)
-		(instances
-			(project "meca_extension_2026"
-				(path "/f6dc6b20-ab52-4b2b-893a-1fb4f3ec4277/067947e6-d018-482f-a78c-eeb83d8dcdcb"
-					(reference "J8")
-					(unit 1)
-				)
-				(path "/f6dc6b20-ab52-4b2b-893a-1fb4f3ec4277/2caf5ca5-b8be-49ab-9f25-cabd53014211"
-					(reference "J5")
-					(unit 1)
-				)
-				(path "/f6dc6b20-ab52-4b2b-893a-1fb4f3ec4277/a1cde7f5-363d-4f36-b502-090ba61d1d03"
-					(reference "J11")
-					(unit 1)
-				)
-				(path "/f6dc6b20-ab52-4b2b-893a-1fb4f3ec4277/cd773c3d-c05b-4eb4-90a6-abf942da4e0b"
-					(reference "J2")
-					(unit 1)
-				)
-			)
-		)
-	)
-	(symbol
 		(lib_id "cocotter_resistors:R_10k_0603_1%")
 		(at 66.04 46.99 0)
@@
 	)
 	(symbol
-		(lib_id "cocotter_connectors:feetech_servo")
-		(at 246.38 35.56 180)
-		(unit 1)
-		(exclude_from_sim no)
-		(in_bom yes)
-		(on_board yes)
-		(dnp no)
-		(fields_autoplaced yes)
-		(property "Reference" "J20"
-			(at 251.206 42.164 0)
-			(effects
-				(font
-					(size 1.27 1.27)
-				)
-				(hide yes)
-			)
-		)
-		(property "Value" "5264-3P"
-			(at 246.38 35.56 0)
-			(effects
-				(font
-					(size 1.27 1.27)
-				)
-				(hide yes)
-			)
-		)
-		(property "Footprint" "cocotter_connectors:5264-3P"
-			(at 246.38 35.56 0)
-			(effects
-				(font
-					(size 1.27 1.27)
-				)
-				(hide yes)
-			)
-		)
-		(property "Datasheet" ""
-			(at 246.38 35.56 0)
-			(effects
-				(font
-					(size 1.27 1.27)
-				)
-				(hide yes)
-			)
-		)
-		(property "Description" ""
-			(at 246.38 35.56 0)
-			(effects
-				(font
-					(size 1.27 1.27)
-				)
-				(hide yes)
-			)
-		)
-		(property "JLC" "C49023819"
-			(at 246.38 35.56 0)
-			(effects
-				(font
-					(size 1.27 1.27)
-				)
-				(hide yes)
-			)
-		)
-		(pin "3"
-		)
-		(pin "2"
-		)
-		(pin "1"
-		)
-		(instances
-			(project "meca_extension_2026"
-				(path "/f6dc6b20-ab52-4b2b-893a-1fb4f3ec4277/067947e6-d018-482f-a78c-eeb83d8dcdcb"
-					(reference "J22")
-					(unit 1)
-				)
-				(path "/f6dc6b20-ab52-4b2b-893a-1fb4f3ec4277/2caf5ca5-b8be-49ab-9f25-cabd53014211"
-					(reference "J21")
-					(unit 1)
-				)
-				(path "/f6dc6b20-ab52-4b2b-893a-1fb4f3ec4277/a1cde7f5-363d-4f36-b502-090ba61d1d03"
-					(reference "J23")
-					(unit 1)
-				)
-				(path "/f6dc6b20-ab52-4b2b-893a-1fb4f3ec4277/cd773c3d-c05b-4eb4-90a6-abf942da4e0b"
-					(reference "J20")
-					(unit 1)
-				)
-			)
-		)
-	)
-	(symbol
 		(lib_id "cocotter_diodes:DSK34")
 		(at 80.01 74.93 270)
@@
 					(unit 1)
 				)
+			)
+		)
+	)
+	(symbol
+		(lib_id "cocotter_connectors:feetech_servo-V")
+		(at 246.38 35.56 180)
+		(unit 1)
+		(exclude_from_sim no)
+		(in_bom yes)
+		(on_board yes)
+		(dnp no)
+		(fields_autoplaced yes)
+		(property "Reference" "J17"
+			(at 251.206 42.164 0)
+			(effects
+				(font
+					(size 1.27 1.27)
+				)
+				(hide yes)
+			)
+		)
+		(property "Value" "5267-3P"
+			(at 246.38 35.56 0)
+			(effects
+				(font
+					(size 1.27 1.27)
+				)
+				(hide yes)
+			)
+		)
+		(property "Footprint" "cocotter_connectors:5267-3P"
+			(at 246.38 35.56 0)
+			(effects
+				(font
+					(size 1.27 1.27)
+				)
+				(hide yes)
+			)
+		)
+		(property "Datasheet" ""
+			(at 246.38 35.56 0)
+			(effects
+				(font
+					(size 1.27 1.27)
+				)
+				(hide yes)
+			)
+		)
+		(property "Description" ""
+			(at 246.38 35.56 0)
+			(effects
+				(font
+					(size 1.27 1.27)
+				)
+				(hide yes)
+			)
+		)
+		(property "JLC" "C49023819"
+			(at 246.38 35.56 0)
+			(effects
+				(font
+					(size 1.27 1.27)
+				)
+				(hide yes)
+			)
+		)
+		(pin "3"
+		)
+		(pin "1"
+		)
+		(pin "2"
+		)
+		(instances
+			(project ""
+				(path "/f6dc6b20-ab52-4b2b-893a-1fb4f3ec4277/067947e6-d018-482f-a78c-eeb83d8dcdcb"
+					(reference "J19")
+					(unit 1)
+				)
+				(path "/f6dc6b20-ab52-4b2b-893a-1fb4f3ec4277/2caf5ca5-b8be-49ab-9f25-cabd53014211"
+					(reference "J18")
+					(unit 1)
+				)
+				(path "/f6dc6b20-ab52-4b2b-893a-1fb4f3ec4277/a1cde7f5-363d-4f36-b502-090ba61d1d03"
+					(reference "J20")
+					(unit 1)
+				)
+				(path "/f6dc6b20-ab52-4b2b-893a-1fb4f3ec4277/cd773c3d-c05b-4eb4-90a6-abf942da4e0b"
+					(reference "J17")
+					(unit 1)
+				)
