File: elec/hw/cartes/picotter_2026/power.kicad_sch (KiCad schematic)
At the start: 74 parts, among them J20 2-1445055-3, Q1 DMP2065UFDB, U6 LV14340DDAR, U7 LV14340DDAR, U8 LV14340DDAR

Commit message: pictotter: schematic fixes after review. New prelayout proposition
Parts:
- removed J20: 2-1445055-3, cocotter_connectors:2-1445055-3, symbol cocotter_connectors:2-1445055-3
- added D13: DSK34, cocotter_diodes:D_SOD-123, symbol cocotter_diodes:DSK34
- added J19: 2-1445051-4, cocotter_connectors:2-1445051-4, symbol cocotter_connectors:2-1445051-4
- added Q19: BSS84, cocotter_transistors:SOT-23-3, symbol cocotter_transistors:BSS84
- added Q20: 2N7002, cocotter_transistors:SOT-23-3, symbol cocotter_transistors:2N7002
- added R71, R72, R73: 100k, cocotter_resistor:r0603_reflow, symbol cocotter_resistors:R_100k_0603_1%
- added R74: 2k2 1%, cocotter_resistor:r0603_reflow, symbol cocotter_resistors:R_2k2_0603_1%
- added R75: 10k 1%, cocotter_resistor:r0603_reflow, symbol cocotter_resistors:R_10k_0603_1%
Connections:
- net +3.3V: now also D13.1 (K)
- net +BATT: now also Q19.2 (S), R71.1
- net GND: now also J19.1, J19.2, Q20.2 (S), R73.2, R74.2
- net at D1.2 (A): now also J19.3, J19.4
- new net: Q19.1 (G), R71.2, R72.1
- new net: Q20.3 (D), R72.2
- new net: Q19.3 (D), R75.1
- new net ena_vbatt_meas_3v3: Q20.1 (G), R73.1
- new net vbatt_meas_3v3: D13.2 (A), R74.1, R75.2

Commit message: picotter: layout almost done (need seriphraphy + layout cleanup)
Parts:
- removed J19: 2-1445051-4, cocotter_connectors:2-1445051-4, symbol cocotter_connectors:2-1445051-4
- removed Q1: DMP2065UFDB, symbol cocotter_transistors:DMP2008UFG-7
- added J20: 3-794630-4, cocotter_connectors:3-794630-4, symbol cocotter_connectors:3-794630-4
- added Q1: PJQ4465AP-AU_R2_000A1, cocotter_transistors:Diodes_PowerDI3333-8, symbol cocotter_transistors:PJQ4465AP-AU_R2_000A1
Connections:
- net +3.3V: now also Q1.1 (S), Q1.2 (S), Q1.3 (S)
- net GND: now also J20.1, J20.2
- net lidar_ena_3v3: now also Q1.4 (G)
- net lidar_pwr_3v3: now also Q1.5 (D)
- net at D1.2 (A): now also J20.3, J20.4
- removed net en_5v: R21.2, R22.1, R23.2, R24.1, R25.2, R26.1, U6.3 (EN), U7.3 (EN), U8.3 (EN)
- new net: R23.2, R24.1, U7.3 (EN)
- new net: R21.2, R22.1, U6.3 (EN)
- new net: R25.2, R26.1, U8.3 (EN)
Changed lines of the file:
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@@
 	(wire
 		(pts
-			(xy 24.13 48.26) (xy 22.86 48.26)
-		)
-		(stroke
-			(width 0)
-			(type default)
-		)
-	)
-	(wire
-		(pts
 			(xy 57.15 105.41) (xy 64.77 105.41)
 		)
@@
 	(wire
 		(pts
+			(xy 12.7 48.26) (xy 12.7 45.72)
+		)
+		(stroke
+			(width 0)
+			(type default)
+		)
+	)
+	(wire
+		(pts
 			(xy 242.57 134.62) (xy 256.54 134.62)
 		)
@@
 	(wire
 		(pts
+			(xy 12.7 48.26) (xy 24.13 48.26)
+		)
+		(stroke
+			(width 0)
+			(type default)
+		)
+	)
+	(wire
+		(pts
 			(xy 157.48 129.54) (xy 158.75 129.54)
 		)
@@
 	(wire
 		(pts
+			(xy 12.7 43.18) (xy 12.7 40.64)
+		)
+		(stroke
+			(width 0)
+			(type default)
+		)
+	)
+	(wire
+		(pts
 			(xy 104.14 95.25) (xy 114.3 95.25)
 		)
@@
 	(wire
 		(pts
+			(xy 12.7 40.64) (xy 24.13 40.64)
+		)
+		(stroke
+			(width 0)
+			(type default)
+		)
+	)
+	(wire
+		(pts
 			(xy 256.54 142.24) (xy 256.54 157.48)
 		)
@@
 	(wire
 		(pts
-			(xy 22.86 40.64) (xy 24.13 40.64)
-		)
-		(stroke
-			(width 0)
-			(type default)
-		)
-	)
-	(wire
-		(pts
 			(xy 200.66 36.83) (xy 200.66 52.07)
 		)
@@
 		)
 	)
-	(label "en_5v"
-		(at 121.92 90.17 0)
-		(effects
-			(font
-				(size 1.27 1.27)
-			)
-			(justify left bottom)
-		)
-	)
-	(label "en_5v"
-		(at 123.19 36.83 0)
-		(effects
-			(font
-				(size 1.27 1.27)
-			)
-			(justify left bottom)
-		)
-	)
-	(label "en_5v"
-		(at 123.19 142.24 0)
-		(effects
-			(font
-				(size 1.27 1.27)
-			)
-			(justify left bottom)
-		)
-	)
 	(hierarchical_label "vbatt_meas_3v3"
 		(shape output)
@@
 	)
 	(symbol
-		(lib_id "cocotter_connectors:2-1445051-4")
-		(at 19.05 44.45 0)
+		(lib_id "cocotter_capacitors:C_22µF_16V_1206_X5R")
+		(at 227.33 86.36 0)
 		(unit 1)
 		(exclude_from_sim no)
@@
 		(on_board yes)
 		(dnp no)
-		(property "Reference" "J19"
-			(at 16.764 38.1 0)
+		(fields_autoplaced yes)
+		(property "Reference" "C58"
+			(at 231.14 85.0899 0)
 			(effects
 				(font
 					(size 1.27 1.27)
 				)
+				(justify left)
 			)
 		)
-		(property "Value" "2-1445051-4"
-			(at 19.812 51.308 0)
+		(property "Value" "22µF 16V"
+			(at 231.14 87.6299 0)
 			(effects
 				(font
 					(size 1.27 1.27)
 				)
+				(justify left)
 			)
 		)
-		(property "Footprint" "cocotter_connectors:2-1445051-4"
-			(at 15.24 41.91 0)
+		(property "Footprint" "cocotter_capacitors:C_1206_3216Metric"
+			(at 228.2952 90.17 0)
 			(effects
 				(font
@@
 			)
 		)
-		(property "Datasheet" ""
-			(at 15.24 41.91 0)
+		(property "Datasheet" "~"
+			(at 227.33 86.36 0)
 			(effects
 				(font
@@
 			)
 		)
-		(property "Description" "1x4POS micro Mate'n LOK, through hole, vertical"
-			(at 15.24 41.91 0)
+		(property "Description" "Unpolarized capacitor"
+			(at 227.33 86.36 0)
 			(effects
 				(font
@@
 			)
 		)
-		(property "JLCPCB Part #" "C17631963"
-			(at 19.05 44.45 0)
+		(property "Specification" "10µF 16V X7R 0805 "
+			(at 227.33 86.36 0)
 			(effects
 				(font
@@
 		(pin "2"
 		)
-		(pin "4"
-		)
-		(pin "3"
-		)
 		(instances
-			(project ""
+			(project "picotter_2026"
 				(path "/a7992a71-8976-4fb0-bae5-4423ba97b789/e08b085d-2769-4f05-b184-06b5277552eb"
-					(reference "J19")
+					(reference "C58")
 					(unit 1)
 				)
@@
 	)
 	(symbol
-		(lib_id "cocotter_capacitors:C_22µF_16V_1206_X5R")
-		(at 227.33 86.36 0)
+		(lib_id "cocotter_connectors:3-794630-4")
+		(at 17.78 44.45 0)
 		(unit 1)
 		(exclude_from_sim no)
@@
 		(dnp no)
 		(fields_autoplaced yes)
-		(property "Reference" "C58"
-			(at 231.14 85.0899 0)
+		(property "Reference" "J20"
+			(at 17.4625 36.83 0)
 			(effects
 				(font
 					(size 1.27 1.27)
 				)
-				(justify left)
 			)
 		)
-		(property "Value" "22µF 16V"
-			(at 231.14 87.6299 0)
+		(property "Value" "3-794630-4"
+			(at 17.4625 39.37 0)
 			(effects
 				(font
 					(size 1.27 1.27)
 				)
-				(justify left)
 			)
 		)
-		(property "Footprint" "cocotter_capacitors:C_1206_3216Metric"
-			(at 228.2952 90.17 0)
+		(property "Footprint" "cocotter_connectors:3-794630-4"
+			(at 17.78 44.45 0)
 			(effects
 				(font
@@
 			)
 		)
-		(property "Datasheet" "~"
-			(at 227.33 86.36 0)
+		(property "Datasheet" "https://www.te.com/commerce/DocumentDelivery/DDEController?Action=srchrtrv&DocNm=82181_SOFTSHELL_HIGH_DENSITY&DocType=Catalog%20Section&DocLang=English&DocFormat=pdf&PartCntxt=794618-4"
+			(at 17.78 44.45 0)
 			(effects
 				(font
@@
 			)
 		)
-		(property "Description" "Unpolarized capacitor"
-			(at 227.33 86.36 0)
+		(property "Description" "2x2POS MICRO MNL ASSY, vertical HDR"
+			(at 17.78 44.45 0)
 			(effects
 				(font
@@
 			)
 		)
-		(property "Specification" "10µF 16V X7R 0805 "
-			(at 227.33 86.36 0)
+		(property "JLCPCB Part #" "C5164688"
+			(at 17.78 44.45 0)
 			(effects
 				(font
@@
 			)
 		)
+		(pin "3"
+		)
+		(pin "4"
+		)
 		(pin "1"
 		)
@@
 		)
 		(instances
-			(project "picotter_2026"
+			(project ""
 				(path "/a7992a71-8976-4fb0-bae5-4423ba97b789/e08b085d-2769-4f05-b184-06b5277552eb"
-					(reference "C58")
+					(reference "J20")
 					(unit 1)
 				)
@@
 	)
 	(symbol
+		(lib_id "cocotter_transistors:PJQ4465AP-AU_R2_000A1")
+		(at 92.71 180.34 270)
+		(mirror x)
+		(unit 1)
+		(exclude_from_sim no)
+		(in_bom yes)
+		(on_board yes)
+		(dnp no)
+		(property "Reference" "Q1"
+			(at 92.456 176.784 90)
+			(effects
+				(font
+					(size 1.27 1.27)
+				)
+			)
+		)
+		(property "Value" "PJQ4465AP-AU_R2_000A1"
+			(at 106.426 185.42 90)
+			(effects
+				(font
+					(size 1.27 1.27)
+				)
+			)
+		)
+		(property "Footprint" "cocotter_transistors:Diodes_PowerDI3333-8"
+			(at 92.71 180.34 0)
+			(effects
+				(font
+					(size 1.27 1.27)
+				)
+				(hide yes)
+			)
+		)
+		(property "Datasheet" ""
+			(at 92.71 180.34 0)
+			(effects
+				(font
+					(size 1.27 1.27)
+				)
+				(hide yes)
+			)
+		)
+		(property "Description" "-55℃~+150℃ 1 P-Channel 1.256nF 1.7V@250uA 15A 20W 22nC@10V 55mΩ@4.5V 59pF 60V 87pF P-Channel DFN3333-8 MOSFETs ROHS"
+			(at 92.71 180.34 0)
+			(effects
+				(font
+					(size 1.27 1.27)
+				)
+				(hide yes)
+			)
+		)
+		(property "JLCPCB Part #" "C6147631"
+			(at 92.71 180.34 0)
+			(effects
+				(font
+					(size 1.27 1.27)
+				)
+				(hide yes)
+			)
+		)
+		(pin "1"
+		)
+		(pin "2"
+		)
+		(pin "5"
+		)
+		(pin "4"
+		)
+		(pin "3"
+		)
+		(instances
+			(project ""
+				(path "/a7992a71-8976-4fb0-bae5-4423ba97b789/e08b085d-2769-4f05-b184-06b5277552eb"
+					(reference "Q1")
+					(unit 1)
+				)
+			)
+		)
+	)
+	(symbol
 		(lib_id "power:GND")
 		(at 66.04 157.48 0)
@@
 					(unit 1)
 				)
-			)
-		)
-	)
-	(symbol
-		(lib_id "cocotter_transistors:DMP2008UFG-7")
-		(at 92.71 180.34 270)
-		(mirror x)
-		(unit 1)
-		(exclude_from_sim no)
-		(in_bom yes)
-		(on_board yes)
-		(dnp no)
-		(property "Reference" "Q1"
-			(at 92.71 170.434 90)
-			(effects
-				(font
-					(size 1.27 1.27)
-				)
-			)
-		)
-		(property "Value" "DMP2065UFDB"
-			(at 92.71 172.72 90)
-			(effects
-				(font
-					(size 1.27 1.27)
-				)
-			)
-		)
-		(property "Footprint" ""
-			(at 92.71 180.34 0)
-			(effects
-				(font
-					(size 1.27 1.27)
-				)
-				(hide yes)
-			)
-		)
-		(property "Datasheet" "cocotter_transistors:Diodes_PowerDI3333-8"
-			(at 92.71 180.34 0)
-			(effects
-				(font
-					(size 1.27 1.27)
-				)
-				(hide yes)
-			)
-		)
-		(property "Description" "PMOS, ID MAX -10A @ Vgs=2.5V, 9.8mOhms@Vgs=2.5V, Vgs max 8V, VDS max 20V"
-			(at 92.71 180.34 0)
-			(effects
-				(font
-					(size 1.27 1.27)
-				)
-				(hide yes)
-			)
-		)
-		(property "JLCPCB Part #" "C461052"
-			(at 92.71 180.34 0)
-			(effects
-				(font
-					(size 1.27 1.27)
-				)
-				(hide yes)
-			)
-		)
-		(pin "4"
-		)
-		(pin "2"
-		)
-		(pin "1"
-		)
-		(pin "5"
-		)
-		(pin "3"
-		)
-		(instances
-			(project ""
-				(path "/a7992a71-8976-4fb0-bae5-4423ba97b789/e08b085d-2769-4f05-b184-06b5277552eb"
-					(reference "Q1")
-					(unit 1)
-				)

Commit message: picotter: final layout
Parts:
- C52, C53, C54, C55, C56, C57, C58, C59, C60, C61, C62, C63, C64, C65, C66: Specification 10µF 16V X7R 0805 -> 22µF 16V X7R 0805
