File: elec/hw/cartes/picotter_2026/uc.kicad_sch (KiCad schematic)
At the start: 20 parts, among them J2 Conn_ARM_SWD_TagConnect_TC2030, U1 STM32H562VGTx, Y1 16MHz 9pF

Commit message: pictotter: schematic fixes after review. New prelayout proposition
Connections:
- net vbatt_meas_3v3: now reaches U1.33 (PC4)
- net ena_vbatt_meas_3v3: now reaches U1.34 (PC5)
- no-connect marks 37 -> 35

Commit message: picotter: layout almost done (need seriphraphy + layout cleanup)
Connections:
- net UART_RX_PRG: no longer U1.68 (PA9)
- net UART_TX_PRG: now also U1.68 (PA9)
- net ena_vbatt_meas_3v3: now also U1.5 (PE6); no longer U1.34 (PC5)
- net irq_floor_0_3v3: now also U1.17 (PC2); no longer U1.15 (PC0)
- net irq_floor_240_3v3: now also U1.80 (PC12); no longer U1.17 (PC2)
- net lidar_rx_0_0_3v3: now also U1.55 (PD8); no longer U1.24 (PA1)
- net lidar_rx_0_120_3v3: now also U1.38 (PE7); no longer U1.56 (PD9)
- net lidar_rx_1_120_3v3: now also U1.24 (PA1); no longer U1.61 (PD14)
- net lidar_rx_1_240_3v3: now also U1.62 (PD15); no longer U1.38 (PE7)
- net lidar_tx_0_0_3v3: now also U1.56 (PD9); no longer U1.23 (PA0)
- net lidar_tx_0_120_3v3: now also U1.39 (PE8); no longer U1.55 (PD8)
- net lidar_tx_1_120_3v3: now also U1.23 (PA0); no longer U1.62 (PD15)
- net lidar_tx_1_240_3v3: now also U1.61 (PD14); no longer U1.39 (PE8)
- net +3V3 renamed +3.3V
- no-connect marks 35 -> 34

Commit message: picotter: final layout
Connections:
- no-connect marks 34 -> 36

Commit message: picotter: add led + 8 testpoints
Parts:
- added D5: green, 0603, cocotter_diodes:LED_0603_1608Metric, symbol cocotter_diodes:green_led_0603
- added R54: 1k 1%, cocotter_resistor:r0603_reflow, symbol cocotter_resistors:R_1k_0603_1%
- added TP1, TP2, TP3, TP4, TP5, TP6, TP7, TP8: TestPoint, cocotter_others:testpoint-THT-0.5mm, symbol cocotter_others:TestPoint
Connections:
- net GND: now also D5.C
- net at U1.41 (PE10): now also TP5.1
- net at U1.42 (PE11): now also TP6.1
- net at U1.43 (PE12): now also TP7.1
- net at U1.44 (PE13): now also TP8.1
- net led: now reaches U1.58 (PD11)
- net led: now also R54.1
- net at U1.85 (PD4): now also TP1.1
- net at U1.86 (PD5): now also TP2.1
- net at U1.87 (PD6): now also TP3.1
- net at U1.88 (PD7): now also TP4.1
- new net: D5.A, R54.2
- no-connect marks 36 -> 27
