File: elec/hw/cartes/tricotter/tricotter.kicad_sch (KiCad schematic)
At the start: 12 parts, among them J1 XT60PW-M, J2 XT60PW-M, J3 XT60PW-M, J5 22053041

Commit message: tricotter : reduced from 5 to 3 power channel and added chaining connector
Parts:
- removed H6: MountingHole_Pad_M3, cocotter_others:MountingHole_3.2mm_M3_Pad_Via, symbol cocotter_others:MountingHole_Pad_M3
- removed J3: XT60PW-M, cocotter_connectors:XT60PW-M, symbol cocotter_connectors:XT60PW-M
- added J3: 22053041, cocotter_connectors:22053041, symbol cocotter_connectors:22053041
- J1: now fitted
Connections:
- net +BATT: now also J3.4
- net GND: now also J3.1; no longer D6.C
- net SW_POWER: now also J3.3
- net SW_logical: now also D6.C, J3.2
Other:
- removed sheet channel3
- removed sheet channel4
- moved on the sheet: D6, R38

Commit message: tricotter 2027 schematic
Parts:
- added R5, R6, R7, R8: 1k 1%, cocotter_resistor:r0603_reflow, symbol cocotter_resistors:R_1k_0603_1%
- R38: mouser 603-RC0603FR-10100KL -> (none)
Connections:
- net SW_POWER: now also R5.1, R7.1
- net SW_logical: now also R6.1, R8.1
- new net channel0/SW_LOGICAL: R6.2, R8.2
- new net channel0/SW_POWER: R5.2, R7.2
Other:
- added sheet com (com.kicad_sch)
